File: luminator.kicad_pcb (KiCad board)
At the start: 2 copper layers, 13 parts

Commit message: up
Parts:
- removed Arduino_Mega_Header: Val**, w_conn_misc:arduino_mega_header_inverted
- removed REF** (x2): SN74AHC595N, SN74AHC595N:SN74AHC595N
- removed REF**: TBD62381APG, TBD62381APG:TBD62381APG
- removed REF**: TBD62786APG, TBD62786APG:TBD62786APG
- removed VASCH_STRIP_10x2 (x4): JP***, w_conn_strip:vasch_strip_10x2
- removed VASCH_STRIP_25x2 (x4): JP***, w_conn_strip:vasch_strip_25x2
Routing:
- net (no net): track 500.4 -> 0.00 mm
Other:
- board text removed: "GND"
- board text removed: "Vcc"
- board text removed: "oe"
- board text removed: "rclk"
- board text removed: "ser"
- board text removed: "srclk"
- board text removed: "srclr"

Commit message: asd
Parts:
- added REF**: 1x3 pads, Luminator:1x3 pads, F.Cu at (84.3, 88.1)
- added REF**: TBD62381APG, Luminator:TBD62381APG, F.Cu at (111.1, 43.2)
- added REF**: M HEADER 2x25=50, Luminator:M HEADER 2x25=50 2.54mm, F.Cu at (127.8, 61.2)
- added REF**: 1x10 pads, Luminator:1x10 pads, F.Cu at (84.5, 55.9)
- added REF**: TBD62381APG, Luminator:TBD62381APG, F.Cu at (111.2, 94.8)
- added REF**: SN74AHC595N, Luminator:SN74AHC595N, F.Cu at (96.6, 119.2)
- added REF**: SN74AHC595N, Luminator:SN74AHC595N, F.Cu at (96.5, 42.2)
- added REF**: 8x10k R Array, Luminator:8x10 R Array, F.Cu at (105.7, 117.7)
- added REF**: SN74AHC595N, Luminator:SN74AHC595N, F.Cu at (96.5, 67.6)
- added REF**: TBD62873APG, Luminator:TBD62783APG, F.Cu at (111.2, 120.2)
- added REF**: 8x10k R Array, Luminator:8x10 R Array, F.Cu at (105.7, 40.6)
- added REF**: TBD62873APG, Luminator:TBD62783APG, F.Cu at (111.1, 68.6)
- added REF**: 8x10k R Array, Luminator:8x10 R Array, F.Cu at (105.7, 92.3)
- added REF**: SN74AHC595N, Luminator:SN74AHC595N, F.Cu at (96.6, 93.8)
- added REF**: 8x10k R Array, Luminator:8x10 R Array, F.Cu at (105.7, 66.0)
Routing:
- net (no net): track 0.00 -> 2990.9 mm, vias 0 -> 16
Other:
- board outline added: 60 x 105 mm
- board text added: "+12/24v"
- board text added: "+5v"
- board text added: "1x10 pads"
- board text added: "8x8 Luminator Driver Revision 1.0 By Tyler Bowers"
- board text added: "COLUMNS"
- board text added: "GND"
- board text added: "OE"
- board text added: "RCLK"
- board text added: "ROWS"
- board text added: "SER"
- board text added: "SRCK"
- board text added: "SRCR"
- board text added: "]"
