File: luminator.kicad_sch (KiCad schematic)
At the start: 1 part

Commit message: up
Parts:
- removed J?: Arduino_Mega_Header, symbol w_connectors:Arduino_Mega_Header
- added U?: TBD62783APG, P-DIP18-300-2p54-001_TOS, symbol Luminator:TBD62783APG
- added U? (x2): SN74AHC595N, N16, symbol Luminator:SN74AHC595N
- added U?: TBD62381APG, P-DIP18-300-2p54-001_TOS, symbol Luminator:TBD62381APG
Connections:
- new net: U?.14 (SER), U?.9 (QH_2)
Changed lines of the file:
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@@
 (kicad_sch (version 20211123) (generator eeschema)
   (paper "A4")
-  (symbol (lib_id "w_connectors:Arduino_Mega_Header") (at 60.96 118.11 0) (unit 1)
+  (wire (pts (xy 26.67 48.26) (xy 24.13 48.26))
+    (stroke (width 0) (type default) (color 0 0 0 0))
+  )
+  (wire (pts (xy 24.13 73.66) (xy 26.67 73.66))
+    (stroke (width 0) (type default) (color 0 0 0 0))
+  )
+  (wire (pts (xy 24.13 48.26) (xy 24.13 73.66))
+    (stroke (width 0) (type default) (color 0 0 0 0))
+  )
+  (symbol (lib_id "Luminator:TBD62783APG") (at 72.39 68.58 0) (unit 1)
     (in_bom yes) (on_board yes) (fields_autoplaced)
-    (property "Reference" "J?" (id 0) (at 60.96 82.55 0)
+    (property "Reference" "U?" (id 0) (at 92.71 58.42 0)
+      (effects (font (size 1.524 1.524)) hide)
+    )
+    (property "Value" "TBD62783APG" (id 1) (at 88.9 60.96 0)
       (effects (font (size 1.524 1.524)))
     )
-    (property "Value" "Arduino_Mega_Header" (id 1) (at 60.96 86.36 0)
+    (property "Footprint" "P-DIP18-300-2p54-001_TOS" (id 2) (at 92.71 60.96 0)
+      (effects (font (size 1.524 1.524)) hide)
+    )
+    (property "Datasheet" "" (id 3) (at 72.39 68.58 0)
       (effects (font (size 1.524 1.524)))
     )
-    (property "Footprint" "" (id 2) (at 60.96 118.11 0)
-      (effects (font (size 1.524 1.524)))
-    )
-    (property "Datasheet" "" (id 3) (at 60.96 118.11 0)
-      (effects (font (size 1.524 1.524)))
-    )
+    (pin "1")
     (pin "10")
     (pin "11")
@@
     (pin "17")
     (pin "18")
-    (pin "19")
     (pin "2")
-    (pin "20")
-    (pin "21")
-    (pin "22")
-    (pin "23")
-    (pin "24")
-    (pin "25")
-    (pin "26")
-    (pin "27")
-    (pin "28")
-    (pin "29")
     (pin "3")
-    (pin "30")
-    (pin "31")
-    (pin "32")
-    (pin "33")
-    (pin "34")
-    (pin "35")
-    (pin "36")
-    (pin "37")
-    (pin "38")
-    (pin "39")
     (pin "4")
-    (pin "40")
-    (pin "41")
-    (pin "42")
-    (pin "43")
-    (pin "44")
-    (pin "45")
-    (pin "46")
-    (pin "47")
-    (pin "48")
-    (pin "49")
     (pin "5")
-    (pin "50")
-    (pin "51")
-    (pin "52")
-    (pin "53")
-    (pin "54")
-    (pin "55")
-    (pin "56")
-    (pin "57")
-    (pin "58")
-    (pin "59")
     (pin "6")
-    (pin "60")
-    (pin "61")
-    (pin "62")
-    (pin "63")
-    (pin "64")
-    (pin "65")
-    (pin "66")
-    (pin "67")
-    (pin "68")
-    (pin "69")
     (pin "7")
-    (pin "70")
-    (pin "71")
-    (pin "72")
-    (pin "73")
-    (pin "74")
-    (pin "75")
-    (pin "76")
-    (pin "77")
-    (pin "78")
-    (pin "79")
     (pin "8")
-    (pin "80")
-    (pin "81")
-    (pin "82")
-    (pin "83")
-    (pin "84")
-    (pin "85")
-    (pin "86")
+    (pin "9")
+  )
+  (symbol (lib_id "Luminator:SN74AHC595N") (at 11.43 68.58 0) (unit 1)
+    (in_bom yes) (on_board yes) (fields_autoplaced)
+    (property "Reference" "U?" (id 0) (at 36.83 59.69 0)
+      (effects (font (size 1.524 1.524)) hide)
+    )
+    (property "Value" "SN74AHC595N" (id 1) (at 43.18 60.96 0)
+      (effects (font (size 1.524 1.524)))
+    )
+    (property "Footprint" "N16" (id 2) (at 38.1 62.23 0)
+      (effects (font (size 1.524 1.524)) hide)
+    )
+    (property "Datasheet" "" (id 3) (at 59.69 71.12 0)
+      (effects (font (size 1.524 1.524)))
+    )
+    (pin "1")
+    (pin "10")
+    (pin "11")
+    (pin "12")
+    (pin "13")
+    (pin "14")
+    (pin "15")
+    (pin "16")
+    (pin "2")
+    (pin "3")
+    (pin "4")
+    (pin "5")
+    (pin "6")
+    (pin "7")
+    (pin "8")
+    (pin "9")
+  )
+  (symbol (lib_id "Luminator:TBD62381APG") (at 72.39 30.48 0) (unit 1)
+    (in_bom yes) (on_board yes) (fields_autoplaced)
+    (property "Reference" "U?" (id 0) (at 82.55 21.59 0)
+      (effects (font (size 1.524 1.524)) hide)
+    )
+    (property "Value" "TBD62381APG" (id 1) (at 88.9 22.86 0)
+      (effects (font (size 1.524 1.524)))
+    )
+    (property "Footprint" "P-DIP18-300-2p54-001_TOS" (id 2) (at 92.71 22.86 0)
+      (effects (font (size 1.524 1.524)) hide)
+    )
+    (property "Datasheet" "" (id 3) (at 72.39 30.48 0)
+      (effects (font (size 1.524 1.524)))
+    )
+    (pin "1")
+    (pin "10")
+    (pin "11")
+    (pin "12")
+    (pin "13")
+    (pin "14")
+    (pin "15")
+    (pin "16")
+    (pin "17")
+    (pin "18")
+    (pin "2")
+    (pin "3")
+    (pin "4")
+    (pin "5")
+    (pin "6")
+    (pin "7")
+    (pin "8")
+    (pin "9")
+  )
+  (symbol (lib_id "Luminator:SN74AHC595N") (at 11.43 30.48 0) (unit 1)
+    (in_bom yes) (on_board yes) (fields_autoplaced)
+    (property "Reference" "U?" (id 0) (at 36.83 21.59 0)
+      (effects (font (size 1.524 1.524)) hide)
+    )
+    (property "Value" "SN74AHC595N" (id 1) (at 43.18 22.86 0)
+      (effects (font (size 1.524 1.524)))
+    )
+    (property "Footprint" "N16" (id 2) (at 38.1 24.13 0)
+      (effects (font (size 1.524 1.524)) hide)
+    )
+    (property "Datasheet" "" (id 3) (at 59.69 33.02 0)
+      (effects (font (size 1.524 1.524)))
+    )
+    (pin "1")
+    (pin "10")
+    (pin "11")
+    (pin "12")
+    (pin "13")
+    (pin "14")
+    (pin "15")
+    (pin "16")
+    (pin "2")
+    (pin "3")
+    (pin "4")
+    (pin "5")
+    (pin "6")
+    (pin "7")
+    (pin "8")
     (pin "9")
   )
@@
   )
   (symbol_instances
-    (path "/baae2c4f-f9e1-4f89-8345-b4655827e8b7"
-      (reference "J?") (unit 1) (value "Arduino_Mega_Header") (footprint "")
+    (path "/01edcc3c-c5fa-4dd7-82f0-8c720850f2b7"
+      (reference "U?") (unit 1) (value "TBD62783APG") (footprint "P-DIP18-300-2p54-001_TOS")
+    )
+    (path "/1f18d333-e45f-41f3-9b3a-d6aa8ca0bd1e"
+      (reference "U?") (unit 1) (value "SN74AHC595N") (footprint "N16")
+    )
+    (path "/da705b04-79d8-4f23-8082-57717462aee1"
+      (reference "U?") (unit 1) (value "TBD62381APG") (footprint "P-DIP18-300-2p54-001_TOS")
+    )
+    (path "/f89dad4a-047f-4db3-b2bf-97c8dbccd2c2"
+      (reference "U?") (unit 1) (value "SN74AHC595N") (footprint "N16")
     )
   )

Commit message: up
Parts:
- added A?: Arduino Mega, ARDUINO_A000067, symbol Luminator:Arduino Mega
- added C? (x2): 0.1uF, symbol Device:C
- added RN? (x2): 8x10k ResistorNet_vert, Resistor_THT:R_Array_SIP10, symbol Luminator:8xResistorNet_vert
Connections:
- net at U?.1 (I1): now also U?.15 (QA), RN?.2 (R1) (x2)
- net GND: now reaches U?.10 (GND)
- net GND: now also U?.8 (GND), U?.8 (GND), U?.9 (GND), C?.1, C?.1, RN?.1 (common), RN?.1 (common)
- net at U?.2 (I2): now also U?.1 (QB), RN?.3 (R2) (x2)
- net at U?.3 (I3): now also U?.2 (QC), RN?.4 (R3) (x2)
- net at U?.4 (I4): now also U?.3 (QD), RN?.5 (R4) (x2)
- net at U?.5 (I5): now also U?.4 (QE), RN?.6 (R5) (x2)
- net at U?.6 (I6): now also U?.5 (QF), RN?.7 (R6) (x2)
- net at U?.7 (I7): now also U?.6 (QG), RN?.8 (R7) (x2)
- net at U?.8 (I8): now also U?.7 (QH), RN?.9 (R8) (x2)
- net +1V0: now reaches U?.9 (VCC)
- net +1V0: now also U?.10 (VCC)
- net at U?.10 (*SRCLR): now also U?.10 (*SRCLR), A?.6
- net at U?.11 (SRCLK): now also U?.11 (SRCLK), A?.4
- net at U?.12 (RCLK): now also U?.12 (RCLK), A?.3
- net at U?.13 (*OE): now also U?.13 (*OE), A?.5
- net +5V: now reaches U?.16 (VCCC)
- net +5V: now also U?.16 (VCCC), C?.2, C?.2
- net at U?.14 (SER): now also A?.2

Commit message: asd
Parts:
- added C? (x2): 0.1uF, symbol Device:C
- added RN? (x2): 8x10k ResistorNet_vert, Resistor_THT:R_Array_SIP10, symbol Luminator:8xResistorNet_vert
- added U?: TBD62381APG, P-DIP18-300-2p54-001_TOS, symbol Luminator:TBD62381APG
- added U? (x2): SN74AHC595N, N16, symbol Luminator:SN74AHC595N
- added U?: TBD62783APG, P-DIP18-300-2p54-001_TOS, symbol Luminator:TBD62783APG
Connections:
- net +1V0: now also U?.10 (VCC), U?.9 (VCC)
- net +5V: now also C?.2, C?.2, U?.16 (VCCC), U?.16 (VCCC)
- net GND: now also C?.1, C?.1, RN?.1 (common), RN?.1 (common), U?.10 (GND), U?.8 (GND), U?.8 (GND), U?.9 (GND)
- net at A?.10: now also U?.13 (*OE), U?.13 (*OE)
- net at A?.11: now also U?.10 (*SRCLR), U?.10 (*SRCLR)
- net at A?.7: now also U?.14 (SER)
- net at A?.8: now also U?.12 (RCLK), U?.12 (RCLK)
- net at A?.9: now also U?.11 (SRCLK), U?.11 (SRCLK)
- new net: RN?.2 (R1), U?.1 (I1), U?.15 (QA) (x2)
- new net: RN?.3 (R2), U?.1 (QB), U?.2 (I2) (x2)
- new net: RN?.4 (R3), U?.2 (QC), U?.3 (I3) (x2)
- new net: RN?.5 (R4), U?.3 (QD), U?.4 (I4) (x2)
- new net: RN?.6 (R5), U?.4 (QE), U?.5 (I5) (x2)
- new net: RN?.7 (R6), U?.5 (QF), U?.6 (I6) (x2)
- new net: RN?.8 (R7), U?.6 (QG), U?.7 (I7) (x2)
- new net: RN?.9 (R8), U?.7 (QH), U?.8 (I8) (x2)
- new net: U?.14 (SER), U?.9 (QH_2)
