File: 8x8 board/luminator.kicad_sch (KiCad schematic)
At the start: 17 parts

Commit message: asd
Connections:
- net +1V0: no longer U?.10 (VCC), U?.10 (VCC)
- net +5V: now also U?.10 (VCC), U?.10 (VCC)
Changed lines of the file:
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@@
     (pin "VIN")
+  )
+  (symbol (lib_id "power:+5V") (at 165.1 67.945 0) (unit 1)
+    (in_bom yes) (on_board yes) (fields_autoplaced)
+    (property "Reference" "#PWR?" (id 0) (at 165.1 71.755 0)
+      (effects (font (size 1.27 1.27)) hide)
+    )
+    (property "Value" "+5V" (id 1) (at 165.1 62.23 0))
+    (property "Footprint" "" (id 2) (at 165.1 67.945 0)
+      (effects (font (size 1.27 1.27)) hide)
+    )
+    (property "Datasheet" "" (id 3) (at 165.1 67.945 0)
+      (effects (font (size 1.27 1.27)) hide)
+    )
+    (pin "1")
   )
   (symbol (lib_id "power:+5V") (at 89.535 31.115 0) (unit 1)
@@
     )
     (property "Datasheet" "" (id 3) (at 89.535 145.415 0)
-      (effects (font (size 1.27 1.27)) hide)
-    )
-    (pin "1")
-  )
-  (symbol (lib_id "Luminator:+12V-24V") (at 165.1 67.945 0) (unit 1)
-    (in_bom yes) (on_board yes) (fields_autoplaced)
-    (property "Reference" "#PWR?" (id 0) (at 165.1 71.755 0)
-      (effects (font (size 1.27 1.27)) hide)
-    )
-    (property "Value" "+12V-24V" (id 1) (at 165.1 62.23 0))
-    (property "Footprint" "" (id 2) (at 165.1 67.945 0)
-      (effects (font (size 1.27 1.27)) hide)
-    )
-    (property "Datasheet" "" (id 3) (at 165.1 67.945 0)
       (effects (font (size 1.27 1.27)) hide)
     )
@@
     (pin "1")
   )
+  (symbol (lib_id "power:+5V") (at 165.1 182.245 0) (unit 1)
+    (in_bom yes) (on_board yes)
+    (property "Reference" "#PWR?" (id 0) (at 165.1 186.055 0)
+      (effects (font (size 1.27 1.27)) hide)
+    )
+    (property "Value" "+5V" (id 1) (at 165.1 178.689 0))
+    (property "Footprint" "" (id 2) (at 165.1 182.245 0)
+      (effects (font (size 1.27 1.27)) hide)
+    )
+    (property "Datasheet" "" (id 3) (at 165.1 182.245 0)
+      (effects (font (size 1.27 1.27)) hide)
+    )
+    (pin "1")
+  )
   (symbol (lib_id "power:GND") (at 83.185 189.23 0) (unit 1)
     (in_bom yes) (on_board yes) (fields_autoplaced)
@@
     (pin "8")
     (pin "9")
-  )
-  (symbol (lib_id "Luminator:+12V-24V") (at 165.1 182.245 0) (unit 1)
-    (in_bom yes) (on_board yes) (fields_autoplaced)
-    (property "Reference" "#PWR?" (id 0) (at 165.1 186.055 0)
-      (effects (font (size 1.27 1.27)) hide)
-    )
-    (property "Value" "+12V-24V" (id 1) (at 165.1 176.53 0))
-    (property "Footprint" "" (id 2) (at 165.1 182.245 0)
-      (effects (font (size 1.27 1.27)) hide)
-    )
-    (property "Datasheet" "" (id 3) (at 165.1 182.245 0)
-      (effects (font (size 1.27 1.27)) hide)
-    )
-    (pin "1")
   )
   (symbol (lib_id "power:GND") (at 135.255 13.97 0) (unit 1)
@@
       (reference "#PWR?") (unit 1) (value "GND") (footprint "")
     )
+    (path "/49d23c97-da0c-4eaa-9def-a844ba4e55f3"
+      (reference "#PWR?") (unit 1) (value "+5V") (footprint "")
+    )
     (path "/4fce0ccf-6613-4faa-814a-a63dcf151455"
       (reference "#PWR?") (unit 1) (value "+5V") (footprint "")
@@
       (reference "#PWR?") (unit 1) (value "+5V") (footprint "")
     )
-    (path "/7aa09a2f-5955-437b-8095-3453dabe0979"
-      (reference "#PWR?") (unit 1) (value "+12V-24V") (footprint "")
-    )
     (path "/865f7c83-fa5f-4d4d-b26e-f82385cfbdfb"
       (reference "#PWR?") (unit 1) (value "+5V") (footprint "")
@@
       (reference "#PWR?") (unit 1) (value "GND") (footprint "")
     )
+    (path "/a13c7b45-de76-46dc-a885-70bd68734900"
+      (reference "#PWR?") (unit 1) (value "+5V") (footprint "")
+    )
     (path "/a1fd5f95-d840-42fc-ad4d-367ba3a36e1e"
       (reference "#PWR?") (unit 1) (value "GND") (footprint "")
     )
-    (path "/c79ee8da-49f9-41b5-a156-e26a48a2ca05"
-      (reference "#PWR?") (unit 1) (value "+12V-24V") (footprint "")
-    )
     (path "/d7df971b-ad0d-4bd8-809c-7741dfb9f827"
