File: 8x8 board/luminator.kicad_pcb (KiCad board)
At the start: 2 copper layers, 60 x 105 mm, 15 parts

Commit message: asd
Routing:
- net (no net): track 2990.9 -> 2998.7 mm, vias 16 -> 18

Commit message: asd
Parts:
- turned REF** to 180 degrees
Changed lines of the file:
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@@
   )
   (footprint "Luminator:1x10 pads" (layer "F.Cu")
-    (at 84.455 55.88 -90)
-    (fp_text reference "REF**" (at 0 2.25 90) (layer "F.SilkS") hide
+    (at 84.455 55.88 180)
+    (fp_text reference "REF**" (at 0 2.25) (layer "F.SilkS") hide
       (effects (font (size 1 1) (thickness 0.15)))
     )
-    (fp_text value "1x10 pads" (at -0.254 6.223 90) (layer "F.Fab") hide
+    (fp_text value "1x10 pads" (at -0.254 6.223) (layer "F.Fab") hide
       (effects (font (size 1 1) (thickness 0.15)))
     )
@@
     (fp_line (start 1 -12.43) (end 1 12.43) (layer "F.CrtYd") (width 0.05))
     (fp_line (start -1 12.43) (end -1 -12.43) (layer "F.CrtYd") (width 0.05))
-    (pad "1" thru_hole circle (at 0 11.43) (size 1.5 1.5) (drill 0.8) (layers *.Cu *.Mask))
-    (pad "2" thru_hole circle (at 0 8.89) (size 1.5 1.5) (drill 0.8) (layers *.Cu *.Mask))
-    (pad "3" thru_hole circle (at 0 6.35) (size 1.5 1.5) (drill 0.8) (layers *.Cu *.Mask))
-    (pad "4" thru_hole circle (at 0 3.81) (size 1.5 1.5) (drill 0.8) (layers *.Cu *.Mask))
-    (pad "5" thru_hole circle (at 0 1.27) (size 1.5 1.5) (drill 0.8) (layers *.Cu *.Mask))
-    (pad "6" thru_hole circle (at 0 -1.27) (size 1.5 1.5) (drill 0.8) (layers *.Cu *.Mask))
-    (pad "7" thru_hole circle (at 0 -3.81) (size 1.5 1.5) (drill 0.8) (layers *.Cu *.Mask))
-    (pad "8" thru_hole circle (at 0 -6.35) (size 1.5 1.5) (drill 0.8) (layers *.Cu *.Mask))
-    (pad "9" thru_hole circle (at 0 -8.89) (size 1.5 1.5) (drill 0.8) (layers *.Cu *.Mask))
-    (pad "10" thru_hole circle (at 0 -11.43) (size 1.5 1.5) (drill 0.8) (layers *.Cu *.Mask))
+    (pad "1" thru_hole circle (at 0 11.43 270) (size 1.5 1.5) (drill 0.8) (layers *.Cu *.Mask))
+    (pad "2" thru_hole circle (at 0 8.89 270) (size 1.5 1.5) (drill 0.8) (layers *.Cu *.Mask))
+    (pad "3" thru_hole circle (at 0 6.35 270) (size 1.5 1.5) (drill 0.8) (layers *.Cu *.Mask))
+    (pad "4" thru_hole circle (at 0 3.81 270) (size 1.5 1.5) (drill 0.8) (layers *.Cu *.Mask))
+    (pad "5" thru_hole circle (at 0 1.27 270) (size 1.5 1.5) (drill 0.8) (layers *.Cu *.Mask))
+    (pad "6" thru_hole circle (at 0 -1.27 270) (size 1.5 1.5) (drill 0.8) (layers *.Cu *.Mask))
+    (pad "7" thru_hole circle (at 0 -3.81 270) (size 1.5 1.5) (drill 0.8) (layers *.Cu *.Mask))
+    (pad "8" thru_hole circle (at 0 -6.35 270) (size 1.5 1.5) (drill 0.8) (layers *.Cu *.Mask))
+    (pad "9" thru_hole circle (at 0 -8.89 270) (size 1.5 1.5) (drill 0.8) (layers *.Cu *.Mask))
+    (pad "10" thru_hole circle (at 0 -11.43 270) (size 1.5 1.5) (drill 0.8) (layers *.Cu *.Mask))
   )
   (footprint "Luminator:TBD62381APG" (layer "F.Cu")
