File: Final Board/luminator/luminator.kicad_sch (KiCad schematic)
At the start: 132 parts

Commit message: asd
Parts:
- added J?: Board #2 Small Connector, CONN20_D10-ST-BK_SUL, symbol Luminator:SBH11-PBPC-D10-ST-BK
- added J?: Board #3 Small Connector, CONN20_D10-ST-BK_SUL, symbol Luminator:SBH11-PBPC-D10-ST-BK
- added J?: Board #3 Large Connector, CONN_SBH11-PBPC-D25-ST-BK_SUL, symbol Luminator:SBH11-PBPC-D25-ST-BK
- added J?: Board #1 Small Connector, CONN20_D10-ST-BK_SUL, symbol Luminator:SBH11-PBPC-D10-ST-BK
- added J?: Board #4 Small Connector, CONN20_D10-ST-BK_SUL, symbol Luminator:SBH11-PBPC-D10-ST-BK
- added J?: Board #4 Large Connector, CONN_SBH11-PBPC-D25-ST-BK_SUL, symbol Luminator:SBH11-PBPC-D25-ST-BK
- added J?: Board #2 Large Connector, CONN_SBH11-PBPC-D25-ST-BK_SUL, symbol Luminator:SBH11-PBPC-D25-ST-BK
- added J?: Board #1 Large Connector, CONN_SBH11-PBPC-D25-ST-BK_SUL, symbol Luminator:SBH11-PBPC-D25-ST-BK
Connections:
- net COL 1: now also J?.10, J?.10, J?.10, J?.10
- net COL 10: now also J?.16, J?.16, J?.16, J?.16
- net COL 11: now also J?.18, J?.18, J?.18, J?.18
- net COL 12: now also J?.20, J?.20, J?.20, J?.20
- net COL 13: now also J?.22, J?.22, J?.22, J?.22
- net COL 14: now also J?.24, J?.24, J?.24, J?.24
- net COL 15: now also J?.26, J?.26, J?.26, J?.26
- net COL 16: now also J?.28, J?.28, J?.28, J?.28
- net COL 17: now also J?.30, J?.30, J?.30, J?.30
- net COL 18: now also J?.32, J?.32, J?.32, J?.32
- net COL 19: now also J?.34, J?.34, J?.34, J?.34
- net COL 2: now also J?.8, J?.8, J?.8, J?.8
- net COL 20: now also J?.36, J?.36, J?.36, J?.36
- net COL 21: now also J?.37, J?.37, J?.37, J?.37
- net COL 22: now also J?.41, J?.41, J?.41, J?.41
- net COL 23: now also J?.45, J?.45, J?.45, J?.45
- net COL 24: now also J?.47, J?.47, J?.47, J?.47
- net COL 25: now also J?.49, J?.49, J?.49, J?.49
- net COL 26: now also J?.50, J?.50, J?.50, J?.50
- net COL 27: now also J?.48, J?.48, J?.48, J?.48
- net COL 28: now also J?.46, J?.46, J?.46, J?.46
- net COL 3: now also J?.6, J?.6, J?.6, J?.6
- net COL 4: now also J?.4, J?.4, J?.4, J?.4
- net COL 5: now also J?.2, J?.2, J?.2, J?.2
- net COL 6: now also J?.1, J?.1, J?.1, J?.1
- net COL 7: now also J?.3, J?.3, J?.3, J?.3
- net COL 8: now also J?.7, J?.7, J?.7, J?.7
- net COL 9: now also J?.11, J?.11, J?.11, J?.11
- net GND: now also J?.19, J?.19, J?.19, J?.19, J?.20, J?.20, J?.20, J?.20
- net at U?.10 (*SRCLR), U?.10 (*SRCLR), U?.10 (*SRCLR)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: now also A?.6
- net at U?.11 (SRCLK), U?.11 (SRCLK), U?.11 (SRCLK)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: now also A?.4
- net at U?.12 (RCLK), U?.12 (RCLK), U?.12 (RCLK)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: now also A?.3
- net at U?.13 (*OE), U?.13 (*OE), U?.13 (*OE)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: now also A?.5
- net at U?.10 (*SRCLR), U?.10 (*SRCLR), U?.10 (*SRCLR)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: now also A?.11
- net at U?.11 (SRCLK), U?.11 (SRCLK), U?.11 (SRCLK)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: now also A?.9
- net at U?.12 (RCLK), U?.12 (RCLK), U?.12 (RCLK)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: now also A?.8
- net at U?.13 (*OE), U?.13 (*OE), U?.13 (*OE)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: now also A?.10
- net at U?.14 (SER): now also A?.2
- net ESP-01: now reaches A?.14
- net ESP-01: now also A?.15, A?.3V3 (+3V3)
- net RTC Module: now reaches A?.20
- net RTC Module: now also A?.21
- net at A?.7: now also U?.14 (SER)
- new net +12V-24V: J?.17, J?.17, J?.17, J?.17, J?.18, J?.18, J?.18, J?.18
- new net ROW 1 +V: J?.23, J?.23, J?.23, J?.23
- new net ROW 1 GND: J?.21, J?.21, J?.21, J?.21
- new net ROW 10 +V: J?.3, J?.3, J?.3, J?.3
- new net ROW 10 GND: J?.4, J?.4, J?.4, J?.4
- new net ROW 11 +V: J?.5, J?.5, J?.5, J?.5
- new net ROW 11 GND: J?.6, J?.6, J?.6, J?.6
- new net ROW 12 +V: J?.7, J?.7, J?.7, J?.7
- new net ROW 12 GND: J?.8, J?.8, J?.8, J?.8
- new net ROW 13 +V: J?.9, J?.9, J?.9, J?.9
- new net ROW 13 GND: J?.10, J?.10, J?.10, J?.10
- new net ROW 14 +V: J?.11, J?.11, J?.11, J?.11
- new net ROW 14 GND: J?.12, J?.12, J?.12, J?.12
- new net ROW 15 +V: J?.13, J?.13, J?.13, J?.13
- new net ROW 15 GND: J?.14, J?.14, J?.14, J?.14
- new net ROW 16 +V: J?.15, J?.15, J?.15, J?.15
- new net ROW 16 GND: J?.16, J?.16, J?.16, J?.16
- new net ROW 2 +V: J?.27, J?.27, J?.27, J?.27
- new net ROW 2 GND: J?.25, J?.25, J?.25, J?.25
- new net ROW 3 +V: J?.19, J?.19, J?.19, J?.19
- new net ROW 3 GND: J?.17, J?.17, J?.17, J?.17
- new net ROW 4 +V: J?.31, J?.31, J?.31, J?.31
- new net ROW 4 GND: J?.29, J?.29, J?.29, J?.29
- new net ROW 5 +V: J?.15, J?.15, J?.15, J?.15
- new net ROW 5 GND: J?.13, J?.13, J?.13, J?.13
- new net ROW 6 +V: J?.35, J?.35, J?.35, J?.35
- new net ROW 6 GND: J?.33, J?.33, J?.33, J?.33
- new net ROW 7 +V: J?.9, J?.9, J?.9, J?.9
- new net ROW 7 GND: J?.5, J?.5, J?.5, J?.5
- new net ROW 8 +V: J?.43, J?.43, J?.43, J?.43
- new net ROW 8 GND: J?.39, J?.39, J?.39, J?.39
- new net ROW 9 +V: J?.1, J?.1, J?.1, J?.1
- new net ROW 9 GND: J?.2, J?.2, J?.2, J?.2
Other:
- moved on the sheet: RN?

Commit message: asd
Connections:
- net +1V0: now also PS?.1 (+VIN)
- net +5V: now also PS?.3 (+VOUT/GND)
- net GND: now also A?.GND1, PS?.2 (GND/-VOUT)

Commit message: asd
Connections:
- net +1V0: no longer U?.10 (VCC), U?.10 (VCC), U?.10 (VCC), U?.10 (VCC), U?.10 (VCC), U?.10 (VCC), U?.10 (VCC), U?.10 (VCC), U?.10 (VCC), U?.10 (VCC), U?.10 (VCC), U?.10 (VCC), U?.10 (VCC), U?.10 (VCC), U?.10 (VCC), U?.10 (VCC)
- net +5V: now also U?.10 (VCC), U?.10 (VCC), U?.10 (VCC), U?.10 (VCC), U?.10 (VCC), U?.10 (VCC), U?.10 (VCC), U?.10 (VCC), U?.10 (VCC), U?.10 (VCC), U?.10 (VCC), U?.10 (VCC), U?.10 (VCC), U?.10 (VCC), U?.10 (VCC), U?.10 (VCC)

Commit message: asd
Parts:
- removed C? (x20): 0.1uF, symbol Device:C
- removed RN? (x20): 8x10k ResistorNet_vert, Resistor_THT:R_Array_SIP10, symbol Luminator:8xResistorNet_vert
- removed U? (x10): TBD62381APG, P-DIP18-300-2p54-001_TOS, symbol Luminator:TBD62381APG
- removed U? (x20): SN74AHC595N, N16, symbol Luminator:SN74AHC595N
- removed U? (x10): TBD62783APG, P-DIP18-300-2p54-001_TOS, symbol Luminator:TBD62783APG
- added C? (x12): 0.1uF, symbol Device:C
- added RN? (x12): 8x10k ResistorNet_vert, Resistor_THT:R_Array_SIP10, symbol Luminator:8xResistorNet_vert
- added U? (x12): SN74AHC595N, N16, symbol Luminator:SN74AHC595N
- added U? (x6): TBD62381APG, P-DIP18-300-2p54-001_TOS, symbol Luminator:TBD62381APG
- added U? (x6): TBD62783APG, P-DIP18-300-2p54-001_TOS, symbol Luminator:TBD62783APG
- added U?: (no value), symbol Luminator:Temperature_Module
Connections:
- net +3.3V is gone; now on net GND: U?. (VCC)
- net +1V0: now also U?.9 (VCC), U?.9 (VCC), U?.9 (VCC), U?.9 (VCC), U?.9 (VCC), U?.9 (VCC)
- net +5V: now also C?.2, C?.2, C?.2, C?.2, C?.2, C?.2, C?.2, C?.2, C?.2, C?.2, C?.2, C?.2, U?. (Sig), U?.10 (VCC), U?.10 (VCC), U?.10 (VCC), U?.10 (VCC), U?.10 (VCC), U?.10 (VCC), U?.16 (VCCC), U?.16 (VCCC), U?.16 (VCCC), U?.16 (VCCC), U?.16 (VCCC), U?.16 (VCCC), U?.16 (VCCC), U?.16 (VCCC), U?.16 (VCCC), U?.16 (VCCC), U?.16 (VCCC), U?.16 (VCCC)
- net COL 1: no longer U?.14 (O5), U?.14 (O5)
- net COL 2: no longer U?.13 (O6), U?.13 (O6)
- net COL 3: no longer U?.12 (O7), U?.12 (O7)
- net COL 4: no longer U?.11 (O8), U?.11 (O8)
- net GND: now also C?.1, C?.1, C?.1, C?.1, C?.1, C?.1, C?.1, C?.1, C?.1, C?.1, C?.1, C?.1, RN?.1 (common), RN?.1 (common), RN?.1 (common), RN?.1 (common), RN?.1 (common), RN?.1 (common), RN?.1 (common), RN?.1 (common), RN?.1 (common), RN?.1 (common), RN?.1 (common), RN?.1 (common), U?. (Sig), U?.10 (GND), U?.10 (GND), U?.10 (GND), U?.10 (GND), U?.10 (GND), U?.10 (GND), U?.8 (GND), U?.8 (GND), U?.8 (GND), U?.8 (GND), U?.8 (GND), U?.8 (GND), U?.8 (GND), U?.8 (GND), U?.8 (GND), U?.8 (GND), U?.8 (GND), U?.8 (GND), U?.9 (GND), U?.9 (GND), U?.9 (GND), U?.9 (GND), U?.9 (GND), U?.9 (GND)
- net ROW 1: now also U?.18 (O1), U?.18 (O1), U?.18 (O1), U?.18 (O1), U?.18 (O1), U?.18 (O1)
- net ROW 10: now also U?.17 (O2), U?.17 (O2), U?.17 (O2), U?.17 (O2), U?.17 (O2), U?.17 (O2)
- net ROW 11: now also U?.16 (O3), U?.16 (O3), U?.16 (O3), U?.16 (O3), U?.16 (O3), U?.16 (O3)
- net ROW 12: now also U?.15 (O4), U?.15 (O4), U?.15 (O4), U?.15 (O4), U?.15 (O4), U?.15 (O4)
- net ROW 13: now also U?.14 (O5), U?.14 (O5), U?.14 (O5), U?.14 (O5), U?.14 (O5), U?.14 (O5)
- net ROW 14: now also U?.13 (O6), U?.13 (O6), U?.13 (O6), U?.13 (O6), U?.13 (O6), U?.13 (O6)
- net ROW 15: now also U?.12 (O7), U?.12 (O7), U?.12 (O7), U?.12 (O7), U?.12 (O7), U?.12 (O7)
- net ROW 16: now also U?.11 (O8), U?.11 (O8), U?.11 (O8), U?.11 (O8), U?.11 (O8), U?.11 (O8)
- net ROW 2: now also U?.17 (O2), U?.17 (O2), U?.17 (O2), U?.17 (O2), U?.17 (O2), U?.17 (O2)
- net ROW 3: now also U?.16 (O3), U?.16 (O3), U?.16 (O3), U?.16 (O3), U?.16 (O3), U?.16 (O3)
- net ROW 4: now also U?.15 (O4), U?.15 (O4), U?.15 (O4), U?.15 (O4), U?.15 (O4), U?.15 (O4)
- net ROW 5: now also U?.14 (O5), U?.14 (O5), U?.14 (O5), U?.14 (O5), U?.14 (O5), U?.14 (O5)
- net ROW 6: now also U?.13 (O6), U?.13 (O6), U?.13 (O6), U?.13 (O6), U?.13 (O6), U?.13 (O6)
- net ROW 7: now also U?.12 (O7), U?.12 (O7), U?.12 (O7), U?.12 (O7), U?.12 (O7), U?.12 (O7)
- net ROW 8: now also U?.11 (O8), U?.11 (O8), U?.11 (O8), U?.11 (O8), U?.11 (O8), U?.11 (O8)
- net ROW 9: now also U?.18 (O1), U?.18 (O1), U?.18 (O1), U?.18 (O1), U?.18 (O1), U?.18 (O1)
- net at A?.11, U?.10 (*SRCLR), U?.10 (*SRCLR)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: now also U?.10 (*SRCLR), U?.10 (*SRCLR), U?.10 (*SRCLR), U?.10 (*SRCLR), U?.10 (*SRCLR), U?.10 (*SRCLR), U?.10 (*SRCLR), U?.10 (*SRCLR), U?.10 (*SRCLR), U?.10 (*SRCLR), U?.10 (*SRCLR), U?.10 (*SRCLR)
- net at A?.9, U?.11 (SRCLK), U?.11 (SRCLK)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: now also U?.11 (SRCLK), U?.11 (SRCLK), U?.11 (SRCLK), U?.11 (SRCLK), U?.11 (SRCLK), U?.11 (SRCLK), U?.11 (SRCLK), U?.11 (SRCLK), U?.11 (SRCLK), U?.11 (SRCLK), U?.11 (SRCLK), U?.11 (SRCLK)
- net at A?.8, U?.12 (RCLK), U?.12 (RCLK)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: now also U?.12 (RCLK), U?.12 (RCLK), U?.12 (RCLK), U?.12 (RCLK), U?.12 (RCLK), U?.12 (RCLK), U?.12 (RCLK), U?.12 (RCLK), U?.12 (RCLK), U?.12 (RCLK), U?.12 (RCLK), U?.12 (RCLK)
- net at A?.10, U?.13 (*OE), U?.13 (*OE)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: now also U?.13 (*OE), U?.13 (*OE), U?.13 (*OE), U?.13 (*OE), U?.13 (*OE), U?.13 (*OE), U?.13 (*OE), U?.13 (*OE), U?.13 (*OE), U?.13 (*OE), U?.13 (*OE), U?.13 (*OE)
- net Temperature Module: now reaches A?.12
- net at U?.9 (QH_2): now also U?.14 (SER)
- new net: RN?.2 (R1), U?.1 (I1), U?.15 (QA) (x12)
- new net: RN?.3 (R2), U?.1 (QB), U?.2 (I2) (x12)
- new net: RN?.4 (R3), U?.2 (QC), U?.3 (I3) (x12)
- new net: RN?.5 (R4), U?.3 (QD), U?.4 (I4) (x12)
- new net: RN?.6 (R5), U?.4 (QE), U?.5 (I5) (x12)
- new net: RN?.7 (R6), U?.5 (QF), U?.6 (I6) (x12)
- new net: RN?.8 (R7), U?.6 (QG), U?.7 (I7) (x12)
- new net: RN?.9 (R8), U?.7 (QH), U?.8 (I8) (x12)
- new net: U?.14 (SER), U?.9 (QH_2) (x11)
- new net +3V3: U?. (VCC)
- new net Arduino Pin 12: U?. (Sig)
- new net COL 29 (NC): U?.14 (O5), U?.14 (O5)
- new net COL 30 (NC): U?.13 (O6), U?.13 (O6)
- new net COL 31 (NC): U?.12 (O7), U?.12 (O7)
- new net COL 32 (NC): U?.11 (O8), U?.11 (O8)
Other:
- note added: "B1-4: 1-28, 29-32NC"
- note added: "BOARD 1 ROWS"
- note added: "BOARD 2 ROWS"
- note added: "BOARD 3 ROWS"
- note added: "BOARD 4 ROWS"
- note added: "Col "x" connects to col x on board 1, 2, 3, and 4. In other words, columns are synced across boards. Rows are not synced."
- note removed: "B1 1-28 B2 1-4"
- note removed: "B2 5-28 B3 1-8"
- note removed: "B3 9-28 B4 1-12"
- note removed: "B4 13-28"
- note removed: "ROWS"
- company: (none) -> Designed by: Tyler Bowers
- title: (none) -> Luminator 16x112 Driver Board
- moved on the sheet: RN?

Commit message: asd
Parts:
- U1: renamed from U?; value (none) -> Temperature_Module
- gave numbers to parts that had none: 108
