File: Final Board/luminator/luminator.kicad_pcb (KiCad board)
At the start: 2 copper layers, 3 parts

Commit message: asd
Parts:
- added REF**: TBD62381APG, Luminator:TBD62381APG, F.Cu at (64.1, 99.1)
- added REF**: SN74AHC595N, Luminator:SN74AHC595N, F.Cu at (52.2, 98.0)
- added REF**: TBD62873APG, Luminator:TBD62783APG, F.Cu at (64.1, 123.8)
- added REF**: 8x10k R Array, Luminator:8x10 R Array, F.Cu at (60.1, 144.1)
- added REF**: 8x10k R Array, Luminator:8x10 R Array, F.Cu at (60.1, 94.6)
- added REF**: SN74AHC595N, Luminator:SN74AHC595N, F.Cu at (52.2, 73.3)
- added REF**: 0.1uF Ceramic, Luminator:0.1uF Ceramic, F.Cu at (48.3, 46.4)
- added REF**: TBD62873APG, Luminator:TBD62783APG, F.Cu at (64.1, 74.3)
- added REF**: 0.1uF Ceramic, Luminator:0.1uF Ceramic, F.Cu at (48.3, 120.7)
- added REF**: 8x10k R Array, Luminator:8x10 R Array, F.Cu at (60.1, 119.4)
- added REF**: 0.1uF Ceramic, Luminator:0.1uF Ceramic, F.Cu at (48.3, 71.1)
- added REF**: SN74AHC595N, Luminator:SN74AHC595N, F.Cu at (52.2, 122.8)
- added REF**: 0.1uF Ceramic, Luminator:0.1uF Ceramic, F.Cu at (48.3, 95.9)
- moved REF** 0.38 mm to (64.1, 49.5)
- moved REF** 0.38 mm to (60.1, 69.8)
- moved REF** 0.38 mm to (52.2, 48.5)
Routing:
- net (no net): track 0.00 -> 1224.4 mm, vias 0 -> 16

Commit message: asd
Parts:
- removed the REF** at (64.1, 99.1)
- removed the REF** at (52.2, 98.0)
- removed the REF** at (64.1, 123.8)
- removed the REF** at (60.1, 144.1)
- removed the REF** at (48.3, 120.7)
- removed the REF** at (60.1, 119.4)
- removed the REF** at (52.2, 122.8)
- removed the REF** at (48.3, 95.9)
- added REF**: SN74AHC595N, Luminator:SN74AHC595N, F.Cu at (78.9, 68.8)
- added REF**: SN74AHC595N, Luminator:SN74AHC595N, F.Cu at (78.9, 19.3)
- added REF**: 8x10k R Array, Luminator:8x10 R Array, F.Cu at (86.7, 40.6)
- added REF**: 8x10k R Array, Luminator:8x10 R Array, F.Cu at (86.7, 114.9)
- added REF**: TBD62381APG, Luminator:TBD62381APG, F.Cu at (90.8, 20.3)
- added REF**: 0.1uF Ceramic, Luminator:0.1uF Ceramic, F.Cu at (75.0, 66.7)
- added REF**: TBD62873APG, Luminator:TBD62783APG, F.Cu at (90.8, 94.6)
- added REF**: M HEADER 2x10=20, Luminator:M HEADER 2x10=20 2.54mm, F.Cu at (240.0, 59.7)
- added REF**: TBD62381APG, Luminator:TBD62381APG, F.Cu at (90.8, 69.8)
- added REF**: 0.1uF Ceramic, Luminator:0.1uF Ceramic, F.Cu at (75.0, 17.1)
- added REF**: SN74AHC595N, Luminator:SN74AHC595N, F.Cu at (78.9, 44.1)
- added REF**: M HEADER 2x10=20, Luminator:M HEADER 2x10=20 2.54mm, F.Cu at (239.4, 99.1)
- added REF**: M HEADER 2x25=50, Luminator:M HEADER 2x25=50 2.54mm, F.Cu at (183.5, 100.3)
- added REF**: TBD62873APG, Luminator:TBD62783APG, F.Cu at (64.1, 94.6)
- added REF**: 0.1uF Ceramic, Luminator:0.1uF Ceramic, F.Cu at (75.0, 91.4)
- added REF**: M HEADER 2x25=50, Luminator:M HEADER 2x25=50 2.54mm, F.Cu at (149.2, 100.3)
- added REF**: 8x10k R Array, Luminator:8x10 R Array, F.Cu at (86.7, 65.4)
- added REF**: M HEADER 2x10=20, Luminator:M HEADER 2x10=20 2.54mm, F.Cu at (239.4, 80.0)
- added REF**: 0.1uF Ceramic, Luminator:0.1uF Ceramic, F.Cu at (48.3, 66.7)
- added REF**: SN74AHC595N, Luminator:SN74AHC595N, F.Cu at (52.2, 68.8)
- added REF**: M HEADER 2x25=50, Luminator:M HEADER 2x25=50 2.54mm, F.Cu at (200.7, 100.3)
- added REF**: 8x10k R Array, Luminator:8x10 R Array, F.Cu at (60.1, 90.2)
- added REF**: 8x10k R Array, Luminator:8x10 R Array, F.Cu at (86.7, 90.2)
- added REF**: 0.1uF Ceramic, Luminator:0.1uF Ceramic, F.Cu at (48.3, 91.4)
- added REF**: M HEADER 2x25=50, Luminator:M HEADER 2x25=50 2.54mm, F.Cu at (166.4, 100.3)
- added REF**: SN74AHC595N, Luminator:SN74AHC595N, F.Cu at (78.9, 93.6)
- added REF**: 8x10k R Array, Luminator:8x10 R Array, F.Cu at (60.1, 114.9)
- added REF**: 0.1uF Ceramic, Luminator:0.1uF Ceramic, F.Cu at (75.0, 41.9)
- added REF**: TBD62381APG, Luminator:TBD62381APG, F.Cu at (64.1, 69.8)
- added REF**: M HEADER 2x10=20, Luminator:M HEADER 2x10=20 2.54mm, F.Cu at (240.0, 38.1)
- added REF**: TBD62873APG, Luminator:TBD62783APG, F.Cu at (90.8, 45.1)
- added REF**: SN74AHC595N, Luminator:SN74AHC595N, F.Cu at (52.2, 93.6)
- moved REF** 29.2 mm to (48.3, 41.9)
- moved REF** 29.2 mm to (52.2, 19.3)
- moved REF** 29.2 mm to (64.1, 45.1)
- moved REF** 29.2 mm to (64.1, 20.3)
- moved REF** 29.2 mm to (48.3, 17.1)
- moved REF** 29.2 mm to (60.1, 40.6)
- moved REF** 29.2 mm to (60.1, 65.4)
- moved REF** 29.2 mm to (52.2, 44.1)
Routing:
- net (no net): track 1224.4 -> 4052.9 mm, vias 16 -> 96
Other:
- copper layers 2 -> 4
- board text added: "COL 1-8"
- board text added: "COL 17-24"
- board text added: "COL 25-28(32)"
- board text added: "COL 9-16"
- board text added: "Inner layers 1 and 2 are used for tran array outputs to connectors, outer layers are used for component signals."
- board text added: "TODO: Power to tran array, serial order & conn"

Commit message: asd
Parts:
- removed the REF** at (240.0, 59.7)
- removed the REF** at (239.4, 99.1)
- removed the REF** at (183.5, 100.3)
- removed the REF** at (149.2, 100.3)
- removed the REF** at (239.4, 80.0)
- removed the REF** at (200.7, 100.3)
- removed the REF** at (166.4, 100.3)
- removed the REF** at (240.0, 38.1)
- added REF**: 0.1uF Ceramic, Luminator:0.1uF Ceramic, F.Cu at (338.8, 237.6)
- added REF**: SN74AHC595N, Luminator:SN74AHC595N, F.Cu at (31.5, 176.9)
- added REF**: SN74AHC595N, Luminator:SN74AHC595N, F.Cu at (70.7, 205.2)
- added REF**: 0.1uF Ceramic, Luminator:0.1uF Ceramic, F.Cu at (200.9, 280.0)
- added REF**: 8x10k R Array, Luminator:8x10 R Array, F.Cu at (327.0, 214.1)
- added REF**: M HEADER 2x25=50, Luminator:M HEADER 2x25=50 2.54mm, F.Cu at (308.3, 202.1)
- added REF**: SN74AHC595N, Luminator:SN74AHC595N, F.Cu at (197.0, 277.9)
- added REF**: TBD62873APG, Luminator:TBD62783APG, F.Cu at (240.1, 45.1)
- added REF**: SN74AHC595N, Luminator:SN74AHC595N, F.Cu at (31.5, 201.7)
- added REF**: 0.1uF Ceramic, Luminator:0.1uF Ceramic, F.Cu at (66.8, 227.8)
- added REF**: SN74AHC595N, Luminator:SN74AHC595N, F.Cu at (334.9, 210.7)
- added REF**: SN74AHC595N, Luminator:SN74AHC595N, F.Cu at (252.0, 70.9)
- added REF**: TBD62381APG, Luminator:TBD62381APG, F.Cu at (200.1, 69.8)
- added REF**: TBD62381APG, Luminator:TBD62381APG, F.Cu at (240.1, 69.8)
- added REF**: 8x10k R Array, Luminator:8x10 R Array, F.Cu at (164.2, 49.5)
- added REF**: 8x10k R Array, Luminator:8x10 R Array, F.Cu at (39.4, 223.0)
- added REF**: 0.1uF Ceramic, Luminator:0.1uF Ceramic, F.Cu at (216.0, 122.6)
- added REF**: 8x10k R Array, Luminator:8x10 R Array, F.Cu at (105.3, 276.1)
- added REF**: SN74AHC595N, Luminator:SN74AHC595N, F.Cu at (252.0, 95.6)
- added REF**: 0.1uF Ceramic, Luminator:0.1uF Ceramic, F.Cu at (256.0, 73.0)
- added REF**: M HEADER 2x10=20, Luminator:M HEADER 2x10=20 2.54mm, F.Cu at (210.4, 278.1)
- added REF**: SN74AHC595N, Luminator:SN74AHC595N, F.Cu at (334.9, 161.2)
- added REF**: M HEADER 2x25=50, Luminator:M HEADER 2x25=50 2.54mm, F.Cu at (210.4, 244.5)
- added REF**: 0.1uF Ceramic, Luminator:0.1uF Ceramic, F.Cu at (66.8, 178.3)
- added REF**: TBD62873APG, Luminator:TBD62783APG, F.Cu at (200.1, 45.1)
- added REF**: TBD62381APG, Luminator:TBD62381APG, F.Cu at (280.1, 119.4)
- added REF**: M HEADER 2x10=20, Luminator:M HEADER 2x10=20 2.54mm, F.Cu at (225.5, 120.7)
- added REF**: TBD62873APG, Luminator:TBD62783APG, F.Cu at (185.0, 252.1)
- added REF**: 0.1uF Ceramic, Luminator:0.1uF Ceramic, F.Cu at (200.9, 205.7)
- added REF**: SN74AHC595N, Luminator:SN74AHC595N, F.Cu at (292.1, 46.1)
- added REF**: SN74AHC595N, Luminator:SN74AHC595N, F.Cu at (70.7, 180.5)
- added REF**: 0.1uF Ceramic, Luminator:0.1uF Ceramic, F.Cu at (200.9, 230.5)
- added REF**: 8x10k R Array, Luminator:8x10 R Array, F.Cu at (244.2, 49.5)
- added REF**: M HEADER 2x25=50, Luminator:M HEADER 2x25=50 2.54mm, F.Cu at (145.5, 87.0)
- added REF**: 8x10k R Array, Luminator:8x10 R Array, F.Cu at (39.4, 198.2)
- added REF**: SN74AHC595N, Luminator:SN74AHC595N, F.Cu at (212.0, 120.4)
- added REF**: SN74AHC595N, Luminator:SN74AHC595N, F.Cu at (97.4, 230.0)
- added REF**: TBD62381APG, Luminator:TBD62381APG, F.Cu at (322.9, 184.9)
- added REF**: M HEADER 2x10=20, Luminator:M HEADER 2x10=20 2.54mm, F.Cu at (170.4, 278.1)
- added REF**: SN74AHC595N, Luminator:SN74AHC595N, F.Cu at (197.0, 203.6)
- added REF**: M HEADER 2x25=50, Luminator:M HEADER 2x25=50 2.54mm, F.Cu at (129.7, 243.7)
- added REF**: 0.1uF Ceramic, Luminator:0.1uF Ceramic, F.Cu at (66.8, 252.6)
- added REF**: TBD62873APG, Luminator:TBD62783APG, F.Cu at (280.1, 45.1)
- added REF**: 8x10k R Array, Luminator:8x10 R Array, F.Cu at (327.0, 189.4)
- added REF**: SN74AHC595N, Luminator:SN74AHC595N, F.Cu at (197.0, 253.1)
- added REF**: TBD62873APG, Luminator:TBD62783APG, F.Cu at (322.9, 160.1)
- added REF**: 8x10k R Array, Luminator:8x10 R Array, F.Cu at (327.0, 164.6)
- added REF**: 0.1uF Ceramic, Luminator:0.1uF Ceramic, F.Cu at (66.8, 203.1)
- added REF**: 8x10k R Array, Luminator:8x10 R Array, F.Cu at (189.1, 256.5)
- added REF**: 8x10k R Array, Luminator:8x10 R Array, F.Cu at (244.2, 24.8)
- added REF**: TBD62381APG, Luminator:TBD62381APG, F.Cu at (185.0, 276.9)
- added REF**: 0.1uF Ceramic, Luminator:0.1uF Ceramic, F.Cu at (256.0, 122.6)
- added REF**: 8x10k R Array, Luminator:8x10 R Array, F.Cu at (164.2, 74.3)
- added REF**: SN74AHC595N, Luminator:SN74AHC595N, F.Cu at (292.1, 70.9)
- added REF**: 0.1uF Ceramic, Luminator:0.1uF Ceramic, F.Cu at (216.0, 73.0)
- added REF**: SN74AHC595N, Luminator:SN74AHC595N, F.Cu at (197.0, 228.3)
- added REF**: SN74AHC595N, Luminator:SN74AHC595N, F.Cu at (292.1, 120.4)
- added REF**: SN74AHC595N, Luminator:SN74AHC595N, F.Cu at (252.0, 46.1)
- added REF**: 0.1uF Ceramic, Luminator:0.1uF Ceramic, F.Cu at (93.5, 203.1)
- added REF**: SN74AHC595N, Luminator:SN74AHC595N, F.Cu at (334.9, 235.5)
- added REF**: SN74AHC595N, Luminator:SN74AHC595N, F.Cu at (70.7, 254.8)
- added REF**: TBD62873APG, Luminator:TBD62783APG, F.Cu at (280.1, 94.6)
- added REF**: 8x10k R Array, Luminator:8x10 R Array, F.Cu at (39.4, 247.8)
- added REF**: M HEADER 2x25=50, Luminator:M HEADER 2x25=50 2.54mm, F.Cu at (170.4, 244.5)
- added REF**: SN74AHC595N, Luminator:SN74AHC595N, F.Cu at (172.0, 46.1)
- added REF**: 8x10k R Array, Luminator:8x10 R Array, F.Cu at (244.2, 74.3)
- added REF**: TBD62381APG, Luminator:TBD62381APG, F.Cu at (109.3, 231.0)
- added REF**: 0.1uF Ceramic, Luminator:0.1uF Ceramic, F.Cu at (296.0, 48.3)
- added REF**: TBD62873APG, Luminator:TBD62783APG, F.Cu at (240.1, 94.6)
- added REF**: 8x10k R Array, Luminator:8x10 R Array, F.Cu at (327.0, 139.8)
- added REF**: 0.1uF Ceramic, Luminator:0.1uF Ceramic, F.Cu at (338.8, 163.3)
- added REF**: M HEADER 2x25=50, Luminator:M HEADER 2x25=50 2.54mm, F.Cu at (385.0, 80.0)
- added REF**: M HEADER 2x10=20, Luminator:M HEADER 2x10=20 2.54mm, F.Cu at (185.5, 120.7)
- added REF**: SN74AHC595N, Luminator:SN74AHC595N, F.Cu at (212.0, 70.9)
- added REF**: M HEADER 2x25=50, Luminator:M HEADER 2x25=50 2.54mm, F.Cu at (185.5, 87.0)
- added REF**: 8x10k R Array, Luminator:8x10 R Array, F.Cu at (78.6, 226.6)
- added REF**: TBD62381APG, Luminator:TBD62381APG, F.Cu at (43.4, 177.9)
- added REF**: 0.1uF Ceramic, Luminator:0.1uF Ceramic, F.Cu at (338.8, 212.9)
- added REF**: 8x10k R Array, Luminator:8x10 R Array, F.Cu at (284.2, 99.1)
- added REF**: 0.1uF Ceramic, Luminator:0.1uF Ceramic, F.Cu at (176.0, 97.8)
- added REF**: TBD62873APG, Luminator:TBD62783APG, F.Cu at (109.3, 206.2)
- added REF**: TBD62381APG, Luminator:TBD62381APG, F.Cu at (82.7, 181.5)
- added REF**: 0.1uF Ceramic, Luminator:0.1uF Ceramic, F.Cu at (176.0, 48.3)
- added REF**: 0.1uF Ceramic, Luminator:0.1uF Ceramic, F.Cu at (256.0, 97.8)
- added REF**: 8x10k R Array, Luminator:8x10 R Array, F.Cu at (78.6, 251.3)
- added REF**: SN74AHC595N, Luminator:SN74AHC595N, F.Cu at (172.0, 120.4)
- added REF**: SN74AHC595N, Luminator:SN74AHC595N, F.Cu at (31.5, 226.4)
- added REF**: TBD62873APG, Luminator:TBD62783APG, F.Cu at (82.7, 255.8)
- added REF**: SN74AHC595N, Luminator:SN74AHC595N, F.Cu at (97.4, 254.8)
- added REF**: SN74AHC595N, Luminator:SN74AHC595N, F.Cu at (172.0, 95.6)
- added REF**: 8x10k R Array, Luminator:8x10 R Array, F.Cu at (284.2, 49.5)
- added REF**: TBD62381APG, Luminator:TBD62381APG, F.Cu at (160.1, 119.4)
- added REF**: M HEADER 2x25=50, Luminator:M HEADER 2x25=50 2.54mm, F.Cu at (265.5, 87.0)
- added REF**: TBD62381APG, Luminator:TBD62381APG, F.Cu at (185.0, 227.3)
- added REF**: 0.1uF Ceramic, Luminator:0.1uF Ceramic, F.Cu at (338.8, 188.1)
- added REF**: 0.1uF Ceramic, Luminator:0.1uF Ceramic, F.Cu at (93.5, 178.3)
- added REF**: SN74AHC595N, Luminator:SN74AHC595N, F.Cu at (97.4, 180.5)
- added REF**: TBD62873APG, Luminator:TBD62783APG, F.Cu at (109.3, 255.8)
- added REF**: M HEADER 2x25=50, Luminator:M HEADER 2x25=50 2.54mm, F.Cu at (348.3, 202.1)
- added REF**: 8x10k R Array, Luminator:8x10 R Array, F.Cu at (204.2, 24.8)
- added REF**: 8x10k R Array, Luminator:8x10 R Array, F.Cu at (189.1, 182.2)
- added REF**: 8x10k R Array, Luminator:8x10 R Array, F.Cu at (105.3, 201.8)
- added REF**: 8x10k R Array, Luminator:8x10 R Array, F.Cu at (164.2, 24.8)
- added REF**: TBD62873APG, Luminator:TBD62783APG, F.Cu at (200.1, 94.6)
- added REF**: 8x10k R Array, Luminator:8x10 R Array, F.Cu at (78.6, 201.8)
- added REF**: TBD62381APG, Luminator:TBD62381APG, F.Cu at (109.3, 181.5)
- added REF**: M HEADER 2x10=20, Luminator:M HEADER 2x10=20 2.54mm, F.Cu at (145.5, 120.7)
- added REF**: 8x10k R Array, Luminator:8x10 R Array, F.Cu at (164.2, 99.1)
- added REF**: TBD62381APG, Luminator:TBD62381APG, F.Cu at (280.1, 69.8)
- added REF**: 0.1uF Ceramic, Luminator:0.1uF Ceramic, F.Cu at (216.0, 97.8)
- added REF**: 8x10k R Array, Luminator:8x10 R Array, F.Cu at (204.2, 74.3)
- added REF**: SN74AHC595N, Luminator:SN74AHC595N, F.Cu at (212.0, 46.1)
- added REF**: TBD62381APG, Luminator:TBD62381APG, F.Cu at (43.4, 227.5)
- added REF**: SN74AHC595N, Luminator:SN74AHC595N, F.Cu at (252.0, 120.4)
- added REF**: SN74AHC595N, Luminator:SN74AHC595N, F.Cu at (212.0, 95.6)
- added REF**: SN74AHC595N, Luminator:SN74AHC595N, F.Cu at (31.5, 251.2)
- added REF**: 0.1uF Ceramic, Luminator:0.1uF Ceramic, F.Cu at (200.9, 255.3)
- added REF**: TBD62873APG, Luminator:TBD62783APG, F.Cu at (185.0, 202.6)
- added REF**: 8x10k R Array, Luminator:8x10 R Array, F.Cu at (244.2, 99.1)
- added REF**: M HEADER 2x10=20, Luminator:M HEADER 2x10=20 2.54mm, F.Cu at (348.3, 235.7)
- added REF**: 8x10k R Array, Luminator:8x10 R Array, F.Cu at (39.4, 272.5)
- added REF**: 0.1uF Ceramic, Luminator:0.1uF Ceramic, F.Cu at (216.0, 48.3)
- added REF**: TBD62381APG, Luminator:TBD62381APG, F.Cu at (82.7, 231.0)
- added REF**: M HEADER 2x10=20, Luminator:M HEADER 2x10=20 2.54mm, F.Cu at (308.3, 235.7)
- added REF**: 0.1uF Ceramic, Luminator:0.1uF Ceramic, F.Cu at (176.0, 73.0)
- added REF**: 0.1uF Ceramic, Luminator:0.1uF Ceramic, F.Cu at (176.0, 122.6)
- added REF**: 0.1uF Ceramic, Luminator:0.1uF Ceramic, F.Cu at (27.6, 199.5)
- added REF**: 0.1uF Ceramic, Luminator:0.1uF Ceramic, F.Cu at (27.6, 174.8)
- added REF**: 8x10k R Array, Luminator:8x10 R Array, F.Cu at (105.3, 251.3)
- added REF**: TBD62873APG, Luminator:TBD62783APG, F.Cu at (322.9, 209.7)
- added REF**: 0.1uF Ceramic, Luminator:0.1uF Ceramic, F.Cu at (27.6, 224.3)
- added REF**: 8x10k R Array, Luminator:8x10 R Array, F.Cu at (204.2, 99.1)
- added REF**: 8x10k R Array, Luminator:8x10 R Array, F.Cu at (284.2, 74.3)
- added REF**: TBD62381APG, Luminator:TBD62381APG, F.Cu at (160.1, 69.8)
- added REF**: TBD62873APG, Luminator:TBD62783APG, F.Cu at (82.7, 206.2)
- added REF**: SN74AHC595N, Luminator:SN74AHC595N, F.Cu at (97.4, 205.2)
- added REF**: 0.1uF Ceramic, Luminator:0.1uF Ceramic, F.Cu at (93.5, 252.6)
- added REF**: 0.1uF Ceramic, Luminator:0.1uF Ceramic, F.Cu at (27.6, 249.0)
- added REF**: TBD62381APG, Luminator:TBD62381APG, F.Cu at (322.9, 234.4)
- added REF**: 0.1uF Ceramic, Luminator:0.1uF Ceramic, F.Cu at (296.0, 73.0)
- added REF**: TBD62381APG, Luminator:TBD62381APG, F.Cu at (240.1, 119.4)
- added REF**: 0.1uF Ceramic, Luminator:0.1uF Ceramic, F.Cu at (256.0, 48.3)
- added REF**: 8x10k R Array, Luminator:8x10 R Array, F.Cu at (189.1, 207.0)
- added REF**: 0.1uF Ceramic, Luminator:0.1uF Ceramic, F.Cu at (296.0, 122.6)
- added REF**: 8x10k R Array, Luminator:8x10 R Array, F.Cu at (189.1, 231.8)
- added REF**: 0.1uF Ceramic, Luminator:0.1uF Ceramic, F.Cu at (296.0, 97.8)
- added REF**: SN74AHC595N, Luminator:SN74AHC595N, F.Cu at (334.9, 185.9)
- added REF**: TBD62873APG, Luminator:TBD62783APG, F.Cu at (43.4, 202.7)
- added REF**: M HEADER 2x25=50, Luminator:M HEADER 2x25=50 2.54mm, F.Cu at (225.5, 87.0)
- added REF**: M HEADER 2x10=20, Luminator:M HEADER 2x10=20 2.54mm, F.Cu at (265.5, 120.7)
- added REF**: TBD62873APG, Luminator:TBD62783APG, F.Cu at (43.4, 252.2)
- added REF**: 8x10k R Array, Luminator:8x10 R Array, F.Cu at (284.2, 24.8)
- added REF**: TBD62381APG, Luminator:TBD62381APG, F.Cu at (200.1, 119.4)
- added REF**: 8x10k R Array, Luminator:8x10 R Array, F.Cu at (105.3, 226.6)
- added REF**: TBD62873APG, Luminator:TBD62783APG, F.Cu at (160.1, 45.1)
- added REF**: SN74AHC595N, Luminator:SN74AHC595N, F.Cu at (292.1, 95.6)
- added REF**: M HEADER 2x25=50, Luminator:M HEADER 2x25=50 2.54mm, F.Cu at (262.9, 210.2)
- added REF**: 0.1uF Ceramic, Luminator:0.1uF Ceramic, F.Cu at (93.5, 227.8)
- added REF**: SN74AHC595N, Luminator:SN74AHC595N, F.Cu at (70.7, 230.0)
- added REF**: TBD62873APG, Luminator:TBD62783APG, F.Cu at (160.1, 94.6)
- added REF**: 8x10k R Array, Luminator:8x10 R Array, F.Cu at (204.2, 49.5)
- added REF**: 8x10k R Array, Luminator:8x10 R Array, F.Cu at (78.6, 276.1)
- added REF**: SN74AHC595N, Luminator:SN74AHC595N, F.Cu at (172.0, 70.9)
- added XA**: Arduino_Mega2560_Shield, Luminator:Arduino_Mega2560_Shield, F.Cu at (75.3, 120.0)
- moved REF** 34.6 mm to (94.4, 45.1)
- moved REF** 34.6 mm to (94.4, 119.4)
- moved REF** 34.6 mm to (121.0, 69.8)
- moved REF** 34.6 mm to (94.4, 94.6)
- moved REF** 34.6 mm to (94.4, 69.8)
- moved REF** 34.6 mm to (121.0, 94.6)
- moved REF** 34.6 mm to (121.0, 45.1)
- moved REF** 34.6 mm to (121.0, 119.4)
- moved REF** 34.6 mm to (98.4, 99.1)
- moved REF** 34.6 mm to (109.2, 95.9)
- moved REF** 34.6 mm to (82.6, 71.1)
- moved REF** 34.6 mm to (86.5, 23.7)
- moved REF** 34.6 mm to (98.4, 24.8)
- moved REF** 34.6 mm to (86.5, 73.3)
- moved REF** 34.6 mm to (82.6, 95.9)
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Routing:
- net (no net): track 4052.9 -> 35255.9 mm, vias 96 -> 542
Other:
- board text added: "*"
- board text added: "3 4 1 2"
- board text added: "B1"
- board text added: "COLS"

Commit message: asd
Parts:
- removed the REF** at (200.9, 280.0)
- removed the REF** at (197.0, 277.9)
- removed the REF** at (210.4, 278.1)
- removed the REF** at (210.4, 244.5)
- removed the REF** at (185.0, 252.1)
- removed the REF** at (200.9, 205.7)
- removed the REF** at (200.9, 230.5)
- removed the REF** at (170.4, 278.1)
- removed the REF** at (197.0, 203.6)
- removed the REF** at (197.0, 253.1)
- removed the REF** at (189.1, 256.5)
- removed the REF** at (185.0, 276.9)
- removed the REF** at (197.0, 228.3)
- removed the REF** at (170.4, 244.5)
- removed the REF** at (185.0, 227.3)
- removed the REF** at (189.1, 182.2)
- removed the REF** at (200.9, 255.3)
- removed the REF** at (185.0, 202.6)
- removed the REF** at (189.1, 207.0)
- removed the REF** at (189.1, 231.8)
- moved REF** 0.51 mm to (338.8, 213.4)
- moved REF** 0.38 mm to (338.8, 188.5)
- moved REF** 0.25 mm to (338.8, 163.6)
- moved REF** 0.13 mm to (338.8, 237.7)
Routing:
- net (no net): track 35255.9 -> 31786.1 mm, vias 542 -> 460
Other:
- board text added: "+12/24V"
- board text added: "+5V"
- board text added: "GND"

Commit message: asd
Parts:
- removed the REF** at (252.0, 70.9)
- removed the REF** at (240.1, 69.8)
- removed the REF** at (164.2, 49.5)
- removed the REF** at (216.0, 122.6)
- removed the REF** at (252.0, 95.6)
- removed the REF** at (256.0, 73.0)
- removed the REF** at (200.1, 45.1)
- removed the REF** at (280.1, 119.4)
- removed the REF** at (225.5, 120.7)
- removed the REF** at (292.1, 46.1)
- removed the REF** at (244.2, 49.5)
- removed the REF** at (244.2, 24.8)
- removed the REF** at (212.0, 120.4)
- removed the REF** at (280.1, 45.1)
- removed the REF** at (256.0, 122.6)
- removed the REF** at (164.2, 74.3)
- removed the REF** at (292.1, 70.9)
- removed the REF** at (216.0, 73.0)
- removed the REF** at (292.1, 120.4)
- removed the REF** at (252.0, 46.1)
- removed the REF** at (240.1, 94.6)
- removed the REF** at (280.1, 94.6)
- removed the REF** at (172.0, 46.1)
- removed the REF** at (244.2, 74.3)
- removed the REF** at (296.0, 48.3)
- removed the REF** at (385.0, 80.0)
- removed the REF** at (185.5, 120.7)
- removed the REF** at (212.0, 70.9)
- removed the REF** at (185.5, 87.0)
- removed the REF** at (284.2, 99.1)
- removed the REF** at (176.0, 97.8)
- removed the REF** at (176.0, 48.3)
- removed the REF** at (256.0, 97.8)
- removed the REF** at (172.0, 120.4)
- removed the REF** at (160.1, 119.4)
- removed the REF** at (172.0, 95.6)
- removed the REF** at (284.2, 49.5)
- removed the REF** at (265.5, 87.0)
- removed the REF** at (204.2, 24.8)
- removed the REF** at (164.2, 24.8)
- removed the REF** at (200.1, 94.6)
- removed the REF** at (204.2, 74.3)
- removed the REF** at (145.5, 120.7)
- removed the REF** at (164.2, 99.1)
- removed the REF** at (280.1, 69.8)
- removed the REF** at (216.0, 97.8)
- removed the REF** at (212.0, 46.1)
- removed the REF** at (252.0, 120.4)
- removed the REF** at (244.2, 99.1)
- removed the REF** at (212.0, 95.6)
- removed the REF** at (216.0, 48.3)
- removed the REF** at (176.0, 73.0)
- removed the REF** at (176.0, 122.6)
- removed the REF** at (204.2, 99.1)
- removed the REF** at (284.2, 74.3)
- removed the REF** at (160.1, 69.8)
- removed the REF** at (296.0, 73.0)
- removed the REF** at (240.1, 119.4)
- removed the REF** at (256.0, 48.3)
- removed the REF** at (296.0, 122.6)
- removed the REF** at (296.0, 97.8)
- removed the REF** at (225.5, 87.0)
- removed the REF** at (265.5, 120.7)
- removed the REF** at (284.2, 24.8)
- removed the REF** at (200.1, 119.4)
- removed the REF** at (160.1, 45.1)
- removed the REF** at (292.1, 95.6)
- removed the REF** at (262.9, 210.2)
- removed the REF** at (160.1, 94.6)
- removed the REF** at (204.2, 49.5)
- removed the REF** at (200.1, 69.8)
- removed the REF** at (172.0, 70.9)
- removed the REF** at (240.1, 45.1)
- moved REF** 0.51 mm to (82.6, 70.6)
- moved REF** 0.38 mm to (109.2, 46.0)
- moved REF** 0.38 mm to (82.6, 46.0)
- moved REF** 0.38 mm to (109.2, 95.5)
- moved REF** 0.38 mm to (82.6, 95.5)
- moved REF** 0.25 mm to (82.6, 21.3)
- moved REF** 0.25 mm to (109.2, 70.9)
- moved REF** 0.25 mm to (109.2, 21.3)
Routing:
- net (no net): track 31786.1 -> 15354.9 mm, vias 460 -> 260

Commit message: asd
Parts:
- removed the REF** at (97.4, 254.8)
- removed the REF** at (82.6, 21.3)
- removed the REF** at (93.5, 178.3)
- removed the REF** at (97.4, 180.5)
- removed the REF** at (109.3, 255.8)
- removed the REF** at (105.3, 201.8)
- removed the REF** at (78.6, 201.8)
- removed the REF** at (109.3, 181.5)
- removed the REF** at (82.7, 231.0)
- removed the REF** at (109.2, 21.3)
- removed the REF** at (105.3, 251.3)
- removed the REF** at (97.4, 205.2)
- removed the REF** at (82.7, 206.2)
- removed the REF** at (93.5, 252.6)
- removed the REF** at (105.3, 226.6)
- removed the REF** at (93.5, 227.8)
- removed the REF** at (70.7, 230.0)
- removed the REF** at (78.6, 276.1)
- removed the REF** at (70.7, 205.2)
- removed the REF** at (66.8, 227.8)
- removed the REF** at (105.3, 276.1)
- removed the REF** at (66.8, 178.3)
- removed the REF** at (70.7, 180.5)
- removed the REF** at (145.5, 87.0)
- removed the REF** at (97.4, 230.0)
- removed the REF** at (129.7, 243.7)
- removed the REF** at (66.8, 252.6)
- removed the REF** at (66.8, 203.1)
- removed the REF** at (70.7, 254.8)
- removed the REF** at (109.3, 231.0)
- removed the REF** at (93.5, 203.1)
- removed the REF** at (78.6, 226.6)
- removed the REF** at (109.3, 206.2)
- removed the REF** at (82.7, 181.5)
- removed the REF** at (78.6, 251.3)
- removed the REF** at (82.7, 255.8)
- added REF**: TBD62873APG, Luminator:TBD62783APG, F.Cu at (90.0, 202.7)
- added REF**: 0.1uF Ceramic, Luminator:0.1uF Ceramic, F.Cu at (240.5, 73.4)
- added REF**: 0.1uF Ceramic, Luminator:0.1uF Ceramic, F.Cu at (280.5, 48.5)
- added REF**: TBD62873APG, Luminator:TBD62783APG, F.Cu at (224.7, 94.6)
- added REF**: 8x10k R Array, Luminator:8x10 R Array, F.Cu at (174.2, 252.1)
- added REF**: SN74AHC595N, Luminator:SN74AHC595N, F.Cu at (196.6, 95.6)
- added REF**: 0.1uF Ceramic, Luminator:0.1uF Ceramic, F.Cu at (280.5, 98.8)
- added REF**: 0.1uF Ceramic, Luminator:0.1uF Ceramic, F.Cu at (101.1, 248.7)
- added REF**: SN74AHC595N, Luminator:SN74AHC595N, F.Cu at (182.1, 273.4)
- added REF**: TBD62381APG, Luminator:TBD62381APG, F.Cu at (116.7, 227.5)
- added REF**: TBD62381APG, Luminator:TBD62381APG, F.Cu at (224.7, 119.4)
- added REF**: M HEADER 2x25=50, Luminator:M HEADER 2x25=50 2.54mm, F.Cu at (290.1, 87.0)
- added REF**: SN74AHC595N, Luminator:SN74AHC595N, F.Cu at (276.6, 95.6)
- added REF**: M HEADER 2x25=50, Luminator:M HEADER 2x25=50 2.54mm, F.Cu at (137.1, 240.2)
- added REF**: 8x10k R Array, Luminator:8x10 R Array, F.Cu at (228.7, 74.3)
- added REF**: SN74AHC595N, Luminator:SN74AHC595N, F.Cu at (316.6, 70.9)
- added REF**: SN74AHC595N, Luminator:SN74AHC595N, F.Cu at (182.1, 199.1)
- added REF**: 0.1uF Ceramic, Luminator:0.1uF Ceramic, F.Cu at (320.5, 73.4)
- added REF**: TBD62873APG, Luminator:TBD62783APG, F.Cu at (170.1, 198.1)
- added REF**: 0.1uF Ceramic, Luminator:0.1uF Ceramic, F.Cu at (320.5, 48.5)
- added REF** (x2): M HEADER 2x10=20, Luminator:M HEADER 2x10=20 2.54mm, F.Cu at (290.1, 120.7)
- added REF**: TBD62381APG, Luminator:TBD62381APG, F.Cu at (224.7, 69.8)
- added REF**: 8x10k R Array, Luminator:8x10 R Array, F.Cu at (86.0, 247.8)
- added REF**: 8x10k R Array, Luminator:8x10 R Array, F.Cu at (228.7, 99.1)
- added REF**: TBD62381APG, Luminator:TBD62381APG, F.Cu at (184.7, 69.8)
- added REF**: 8x10k R Array, Luminator:8x10 R Array, F.Cu at (228.7, 49.5)
- added REF**: SN74AHC595N, Luminator:SN74AHC595N, F.Cu at (196.6, 120.4)
- added REF**: 8x10k R Array, Luminator:8x10 R Array, F.Cu at (112.6, 198.2)
- added REF** (x2): M HEADER 2x10=20, Luminator:M HEADER 2x10=20 2.54mm, F.Cu at (210.1, 120.7)
- added REF**: 8x10k R Array, Luminator:8x10 R Array, F.Cu at (308.7, 74.3)
- added REF**: SN74AHC595N, Luminator:SN74AHC595N, F.Cu at (316.6, 95.6)
- added REF**: 8x10k R Array, Luminator:8x10 R Array, F.Cu at (112.6, 223.0)
- added REF**: 8x10k R Array, Luminator:8x10 R Array, F.Cu at (86.0, 198.2)
- added REF**: TBD62381APG, Luminator:TBD62381APG, F.Cu at (264.7, 119.4)
- added REF**: 0.1uF Ceramic, Luminator:0.1uF Ceramic, F.Cu at (200.5, 48.5)
- added REF**: 8x10k R Array, Luminator:8x10 R Array, F.Cu at (174.2, 227.3)
- added REF**: 8x10k R Array, Luminator:8x10 R Array, F.Cu at (308.7, 99.1)
- added REF**: 0.1uF Ceramic, Luminator:0.1uF Ceramic, F.Cu at (74.2, 174.5)
- added REF**: SN74AHC595N, Luminator:SN74AHC595N, F.Cu at (78.1, 201.7)
- added REF**: 8x10k R Array, Luminator:8x10 R Array, F.Cu at (86.0, 272.5)
- added REF**: 8x10k R Array, Luminator:8x10 R Array, F.Cu at (188.7, 24.8)
- added REF**: TBD62381APG, Luminator:TBD62381APG, F.Cu at (170.1, 272.4)
- added REF** (x2): M HEADER 2x10=20, Luminator:M HEADER 2x10=20 2.54mm, F.Cu at (250.1, 120.7)
- added REF**: SN74AHC595N, Luminator:SN74AHC595N, F.Cu at (78.1, 251.2)
- added REF**: M HEADER 2x10=20, Luminator:M HEADER 2x10=20 2.54mm, F.Cu at (170.1, 120.7)
- added REF**: TBD62873APG, Luminator:TBD62783APG, F.Cu at (264.7, 94.6)
- added REF**: 8x10k R Array, Luminator:8x10 R Array, F.Cu at (268.7, 49.5)
- added REF**: TBD62381APG, Luminator:TBD62381APG, F.Cu at (90.0, 227.5)
- added REF**: TBD62873APG, Luminator:TBD62783APG, F.Cu at (304.7, 94.6)
- added REF**: SN74AHC595N, Luminator:SN74AHC595N, F.Cu at (78.1, 226.4)
- added REF**: 0.1uF Ceramic, Luminator:0.1uF Ceramic, F.Cu at (186.0, 201.5)
- added REF**: TBD62873APG, Luminator:TBD62783APG, F.Cu at (304.7, 45.1)
- added REF**: 0.1uF Ceramic, Luminator:0.1uF Ceramic, F.Cu at (186.0, 251.8)
- added REF**: 0.1uF Ceramic, Luminator:0.1uF Ceramic, F.Cu at (101.1, 224.0)
- added REF**: SN74AHC595N, Luminator:SN74AHC595N, F.Cu at (236.6, 95.6)
- added REF**: SN74AHC595N, Luminator:SN74AHC595N, F.Cu at (104.8, 251.2)
- added REF**: SN74AHC595N, Luminator:SN74AHC595N, F.Cu at (78.1, 176.9)
- added REF**: 8x10k R Array, Luminator:8x10 R Array, F.Cu at (268.7, 74.3)
- added REF**: SN74AHC595N, Luminator:SN74AHC595N, F.Cu at (104.8, 201.7)
- added REF**: TBD62873APG, Luminator:TBD62783APG, F.Cu at (184.7, 45.1)
- added REF**: M HEADER 2x25=50, Luminator:M HEADER 2x25=50 2.54mm, F.Cu at (170.1, 87.0)
- added REF**: 8x10k R Array, Luminator:8x10 R Array, F.Cu at (174.2, 177.8)
- added REF**: 8x10k R Array, Luminator:8x10 R Array, F.Cu at (188.7, 49.5)
- added REF**: SN74AHC595N, Luminator:SN74AHC595N, F.Cu at (182.1, 248.7)
- added REF**: SN74AHC595N, Luminator:SN74AHC595N, F.Cu at (276.6, 70.9)
- added REF**: 0.1uF Ceramic, Luminator:0.1uF Ceramic, F.Cu at (74.2, 223.8)
- added REF**: 0.1uF Ceramic, Luminator:0.1uF Ceramic, F.Cu at (74.2, 248.7)
- added REF**: 0.1uF Ceramic, Luminator:0.1uF Ceramic, F.Cu at (240.5, 98.8)
- added REF**: M HEADER 2x25=50, Luminator:M HEADER 2x25=50 2.54mm, F.Cu at (250.1, 87.0)
- added REF**: TBD62381APG, Luminator:TBD62381APG, F.Cu at (116.7, 177.9)
- added REF**: TBD62381APG, Luminator:TBD62381APG, F.Cu at (90.0, 177.9)
- added REF**: SN74AHC595N, Luminator:SN74AHC595N, F.Cu at (196.6, 46.1)
- added REF**: SN74AHC595N, Luminator:SN74AHC595N, F.Cu at (276.6, 120.4)
- added REF**: SN74AHC595N, Luminator:SN74AHC595N, F.Cu at (104.8, 176.9)
- added REF**: 8x10k R Array, Luminator:8x10 R Array, F.Cu at (112.6, 247.8)
- added REF**: TBD62873APG, Luminator:TBD62783APG, F.Cu at (116.7, 252.2)
- added REF**: 8x10k R Array, Luminator:8x10 R Array, F.Cu at (268.7, 24.8)
- added REF**: SN74AHC595N, Luminator:SN74AHC595N, F.Cu at (276.6, 46.1)
- added REF**: 0.1uF Ceramic, Luminator:0.1uF Ceramic, F.Cu at (240.5, 48.5)
- added REF**: TBD62381APG, Luminator:TBD62381APG, F.Cu at (304.7, 119.4)
- added REF**: 0.1uF Ceramic, Luminator:0.1uF Ceramic, F.Cu at (100.9, 199.1)
- added REF**: M HEADER 2x10=20, Luminator:M HEADER 2x10=20 2.54mm, F.Cu at (195.5, 273.7)
- added REF**: TBD62381APG, Luminator:TBD62381APG, F.Cu at (304.7, 69.8)
- added REF**: 0.1uF Ceramic, Luminator:0.1uF Ceramic, F.Cu at (200.5, 98.8)
- added REF**: TBD62873APG, Luminator:TBD62783APG, F.Cu at (90.0, 252.2)
- added REF**: M HEADER 2x25=50, Luminator:M HEADER 2x25=50 2.54mm, F.Cu at (195.5, 240.0)
- added REF**: TBD62873APG, Luminator:TBD62783APG, F.Cu at (170.1, 247.7)
- added REF**: 0.1uF Ceramic, Luminator:0.1uF Ceramic, F.Cu at (185.8, 275.2)
- added REF**: 0.1uF Ceramic, Luminator:0.1uF Ceramic, F.Cu at (280.5, 73.4)
- added REF**: SN74AHC595N, Luminator:SN74AHC595N, F.Cu at (236.6, 70.9)
- added REF**: 0.1uF Ceramic, Luminator:0.1uF Ceramic, F.Cu at (186.0, 226.4)
- added REF**: 8x10k R Array, Luminator:8x10 R Array, F.Cu at (268.7, 99.1)
- added REF**: 8x10k R Array, Luminator:8x10 R Array, F.Cu at (308.7, 49.5)
- added REF**: M HEADER 2x25=50, Luminator:M HEADER 2x25=50 2.54mm, F.Cu at (155.5, 240.0)
- added REF**: 8x10k R Array, Luminator:8x10 R Array, F.Cu at (86.0, 223.0)
- added REF**: SN74AHC595N, Luminator:SN74AHC595N, F.Cu at (196.6, 70.9)
- added REF**: TBD62873APG, Luminator:TBD62783APG, F.Cu at (224.7, 45.1)
- added REF**: SN74AHC595N, Luminator:SN74AHC595N, F.Cu at (182.1, 223.9)
- added REF**: SN74AHC595N, Luminator:SN74AHC595N, F.Cu at (236.6, 46.1)
- added REF**: TBD62381APG, Luminator:TBD62381APG, F.Cu at (170.1, 222.9)
- added REF**: 8x10k R Array, Luminator:8x10 R Array, F.Cu at (188.7, 99.1)
- added REF**: 8x10k R Array, Luminator:8x10 R Array, F.Cu at (188.7, 74.3)
- added REF**: SN74AHC595N, Luminator:SN74AHC595N, F.Cu at (316.6, 120.4)
- added REF**: 0.1uF Ceramic, Luminator:0.1uF Ceramic, F.Cu at (320.5, 98.8)
- added REF**: 0.1uF Ceramic, Luminator:0.1uF Ceramic, F.Cu at (100.9, 174.5)
- added REF**: TBD62873APG, Luminator:TBD62783APG, F.Cu at (116.7, 202.7)
- added REF**: 8x10k R Array, Luminator:8x10 R Array, F.Cu at (228.7, 24.8)
- added REF**: 0.1uF Ceramic, Luminator:0.1uF Ceramic, F.Cu at (74.2, 199.1)
- added REF**: 0.1uF Ceramic, Luminator:0.1uF Ceramic, F.Cu at (200.5, 73.4)
- added REF**: TBD62381APG, Luminator:TBD62381APG, F.Cu at (264.7, 69.8)
- added REF**: TBD62873APG, Luminator:TBD62783APG, F.Cu at (184.7, 94.6)
- added REF**: 8x10k R Array, Luminator:8x10 R Array, F.Cu at (112.6, 272.5)
- added REF**: SN74AHC595N, Luminator:SN74AHC595N, F.Cu at (236.6, 120.4)
- added REF**: M HEADER 2x25=50, Luminator:M HEADER 2x25=50 2.54mm, F.Cu at (210.1, 87.0)
- added REF**: TBD62873APG, Luminator:TBD62783APG, F.Cu at (264.7, 45.1)
- added REF**: M HEADER 2x10=20, Luminator:M HEADER 2x10=20 2.54mm, F.Cu at (155.5, 273.7)
- added REF**: TBD62381APG, Luminator:TBD62381APG, F.Cu at (184.7, 119.4)
- added REF**: SN74AHC595N, Luminator:SN74AHC595N, F.Cu at (316.6, 46.1)
- added REF**: SN74AHC595N, Luminator:SN74AHC595N, F.Cu at (104.8, 226.4)
- added REF**: 8x10k R Array, Luminator:8x10 R Array, F.Cu at (308.7, 24.8)
- added REF**: 8x10k R Array, Luminator:8x10 R Array, F.Cu at (174.2, 202.6)
- moved XA** 28.4 mm to (103.6, 122.1)
- moved REF** 24.8 mm to (134.1, 95.5)
- moved REF** 24.8 mm to (134.1, 70.9)
- moved REF** 24.6 mm to (137.7, 48.5)
- moved REF** 24.6 mm to (137.7, 98.0)
- moved REF** 24.6 mm to (133.8, 46.0)
- moved REF** 24.6 mm to (137.7, 73.3)
- moved REF** 24.6 mm to (137.7, 23.7)
- moved REF** 24.6 mm to (149.7, 74.3)
- moved REF** 24.6 mm to (118.9, 45.1)
- moved REF** 24.6 mm to (123.0, 99.1)
- moved REF** 24.6 mm to (145.6, 69.8)
- moved REF** 24.6 mm to (111.1, 23.7)
- moved REF** 24.6 mm to (123.0, 24.8)
- moved REF** 24.6 mm to (111.1, 73.3)
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Routing:
- net (no net): track 15354.9 -> 35654.2 mm, vias 260 -> 397
Other:
- board outline added: 308.6 x 109.2 mm
- board text added: "B2"
- board text added: "B3"
- board text added: "B4"
