File: Final Board/luminator/luminator.kicad_pcb (KiCad board)
At the start: 4 copper layers, 308.6 x 109.2 mm, 191 parts

Commit message: wasd
Parts:
- added REF**: P78E05, Luminator:P78E05, F.Cu at (40.1, 117.9)
Routing:
- net (no net): track 35654.2 -> 35888.9 mm
Changed lines of the file:
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@@
     (pad "18" thru_hole circle (at 7.62 0) (size 1.227074 1.227074) (drill 0.719074) (layers "*.Cu" "*.Mask"))
   )
+  (footprint "Luminator:P78E05" (layer "F.Cu")
+    (at 40.132 117.856)
+    (attr through_hole)
+    (fp_text reference "REF**" (at -2.925 -6.735) (layer "F.SilkS")
+        (effects (font (size 1 1) (thickness 0.15)))
+    )
+    (fp_text value "P78E05" (at 3.96 3.865) (layer "F.Fab")
+        (effects (font (size 1 1) (thickness 0.15)))
+    )
+    (fp_line (start -5.8 -5.7) (end 5.8 -5.7)
+      (stroke (width 0.127) (type solid)) (layer "F.SilkS"))
+    (fp_line (start -5.8 2.3) (end -5.8 -5.7)
+      (stroke (width 0.127) (type solid)) (layer "F.SilkS"))
+    (fp_line (start 5.8 -5.7) (end 5.8 2.3)
+      (stroke (width 0.127) (type solid)) (layer "F.SilkS"))
+    (fp_line (start 5.8 2.3) (end -5.8 2.3)
+      (stroke (width 0.127) (type solid)) (layer "F.SilkS"))
+    (fp_circle (center -2.54 3) (end -2.44 3)
+      (stroke (width 0.2) (type solid)) (fill none) (layer "F.SilkS"))
+    (fp_line (start -6.05 -5.95) (end 6.05 -5.95)
+      (stroke (width 0.05) (type solid)) (layer "F.CrtYd"))
+    (fp_line (start -6.05 2.55) (end -6.05 -5.95)
+      (stroke (width 0.05) (type solid)) (layer "F.CrtYd"))
+    (fp_line (start 6.05 -5.95) (end 6.05 2.55)
+      (stroke (width 0.05) (type solid)) (layer "F.CrtYd"))
+    (fp_line (start 6.05 2.55) (end -6.05 2.55)
+      (stroke (width 0.05) (type solid)) (layer "F.CrtYd"))
+    (fp_line (start -5.8 -5.7) (end 5.8 -5.7)
+      (stroke (width 0.127) (type solid)) (layer "F.Fab"))
+    (fp_line (start -5.8 2.3) (end -5.8 -5.7)
+      (stroke (width 0.127) (type solid)) (layer "F.Fab"))
+    (fp_line (start 5.8 -5.7) (end 5.8 2.3)
+      (stroke (width 0.127) (type solid)) (layer "F.Fab"))
+    (fp_line (start 5.8 2.3) (end -5.8 2.3)
+      (stroke (width 0.127) (type solid)) (layer "F.Fab"))
+    (fp_circle (center -2.54 3) (end -2.44 3)
+      (stroke (width 0.2) (type solid)) (fill none) (layer "F.Fab"))
+    (pad "1" thru_hole rect (at -2.54 0) (size 1.508 1.508) (drill 1) (layers "*.Cu" "*.Mask"))
+    (pad "2" thru_hole circle (at 0 0) (size 1.508 1.508) (drill 1) (layers "*.Cu" "*.Mask"))
+    (pad "3" thru_hole circle (at 2.54 0) (size 1.508 1.508) (drill 1) (layers "*.Cu" "*.Mask"))
+  )
   (footprint "Luminator:8x10 R Array" (layer "F.Cu")
     (at 308.7443 24.765)
@@
     (fp_arc (start 94.488 -54.864) (mid 96.52 -55.524237) (end 98.552 -54.864)
       (stroke (width 0.15) (type solid)) (layer "B.CrtYd"))
-    (fp_arc (start 99.314 -54.102) (mid 99.650926 -53.532027) (end 99.8728 -52.9082)
+    (fp_arc (start 99.314 -54.102) (mid 99.650928 -53.532028) (end 99.8728 -52.9082)
       (stroke (width 0.15) (type solid)) (layer "B.CrtYd"))
     (fp_circle (center 13.97 -52.07) (end 17.42 -52.07)
@@
     (effects (font (size 1.5 1.5) (thickness 0.3)))
   )
-  (gr_text "+12/24V" (at 100.1395 121.92) (layer "B.Cu")
-    (effects (font (size 1.5 1.5) (thickness 0.3)))
-  )
   (gr_text "COL 17-24" (at 108.966 154.686) (layer "B.Cu")
     (effects (font (size 1.5 1.5) (thickness 0.3)))
@@
     (effects (font (size 1 1) (thickness 0.15)))
   )
-  (gr_text "GND" (at 98.2345 125.095) (layer "Cmts.User")
+  (gr_text "GND" (at 24.257 124.841) (layer "Cmts.User")
     (effects (font (size 1.5 1.5) (thickness 0.3) bold) (justify left bottom))
   )
@@
     (effects (font (size 1.5 1.5) (thickness 0.3) bold) (justify left bottom))
   )
-  (gr_text "+5V" (at 99.8855 126.492) (layer "Cmts.User")
+  (gr_text "+12/24V" (at 26.162 121.666) (layer "Cmts.User")
+    (effects (font (size 1.5 1.5) (thickness 0.3)))
+  )
+  (gr_text "+5V" (at 25.908 126.238) (layer "Cmts.User")
     (effects (font (size 1.5 1.5) (thickness 0.3)))
   )
@@
   (segment (start 174.2005 212.725) (end 170.1365 212.725) (width 0.2) (layer "F.Cu") (net 0))
   (segment (start 157.2895 37.465) (end 158.5595 36.195) (width 0.25) (layer "F.Cu") (net 0))
+  (segment (start 37.592 123.063) (end 37.592 117.856) (width 0.6) (layer "F.Cu") (net 0))
   (segment (start 110.49 76.7715) (end 114.3635 80.645) (width 0.2) (layer "F.Cu") (net 0))
   (segment (start 193.314 78.105) (end 190.012 78.105) (width 0.2) (layer "F.Cu") (net 0))
@@
   (segment (start 314.8022 22.8927) (end 314.8276 22.8673) (width 0.2) (layer "F.Cu") (net 0))
   (segment (start 145.6055 99.06) (end 149.6695 99.06) (width 0.2) (layer "F.Cu") (net 0))
+  (segment (start 37.592 123.063) (end 33.909 123.063) (width 0.6) (layer "F.Cu") (net 0))
   (segment (start 133.9215 101.5365) (end 137.16 101.5365) (width 0.2) (layer "F.Cu") (net 0))
   (segment (start 273.5653 104.14) (end 272.8668 104.14) (width 0.2) (layer "F.Cu") (net 0))
@@
   (segment (start 240.431 81.9785) (end 237.1925 81.9785) (width 0.2) (layer "F.Cu") (net 0))
   (segment (start 168.783 106.68) (end 167.513 107.95) (width 0.25) (layer "F.Cu") (net 0))
+  (segment (start 105.7275 123.063) (end 37.592 123.063) (width 0.6) (layer "F.Cu") (net 0))
   (segment (start 104.2035 177.8635) (end 108.077 181.737) (width 0.2) (layer "F.Cu") (net 0))
   (segment (start 178.7725 253.365) (end 175.4705 253.365) (width 0.2) (layer "F.Cu") (net 0))
@@
   (segment (start 169.2075 200.279) (end 164.719 204.7675) (width 0.25) (layer "In1.Cu") (net 0))
   (segment (start 162.4965 94.488) (end 169.9895 86.995) (width 0.25) (layer "In1.Cu") (net 0))
+  (segment (start 42.672 125.349) (end 33.909 125.349) (width 0.6) (layer "In1.Cu") (net 0))
   (segment (start 226.3675 96.774) (end 219.2655 96.774) (width 0.25) (layer "In1.Cu") (net 0))
   (segment (start 316.992 146.6015) (end 315.2975 144.907) (width 0.2) (layer "In1.Cu") (net 0))
@@
   (segment (start 172.974 73.914) (end 172.974 44.323) (width 0.2) (layer "In1.Cu") (net 0))
   (segment (start 164.9095 31.115) (end 166.1795 29.845) (width 0.25) (layer "In1.Cu") (net 0))
+  (segment (start 42.672 125.349) (end 42.672 117.856) (width 0.6) (layer "In1.Cu") (net 0))
   (segment (start 166.8145 42.545) (end 168.7195 42.545) (width 0.25) (layer "In1.Cu") (net 0))
   (segment (start 138.8745 107.315) (end 140.1445 107.315) (width 0.25) (layer "In1.Cu") (net 0))
@@
   (segment (start 175.895 180.975) (end 176.4665 180.4035) (width 0.25) (layer "In1.Cu") (net 0))
   (segment (start 272.8395 119.4435) (end 275.717 119.4435) (width 0.25) (layer "In1.Cu") (net 0))
+  (segment (start 105.7275 125.349) (end 42.672 125.349) (width 0.6) (layer "In1.Cu") (net 0))
   (segment (start 215.265 40.005) (end 211.455 43.815) (width 0.2) (layer "In1.Cu") (net 0))
   (segment (start 88.138 268.732) (end 88.9 267.97) (width 0.25) (layer "In1.Cu") (net 0))
@@
   (segment (start 112.2045 85.09) (end 112.2045 109.855) (width 0.2) (layer "B.Cu") (net 0))
   (segment (start 252.2093 102.489) (end 251.8283 102.87) (width 0.25) (layer "B.Cu") (net 0))
+  (segment (start 40.132 124.206) (end 33.782 124.206) (width 0.6) (layer "B.Cu") (net 0))
   (segment (start 320.4283 73.132) (end 320.5353 73.025) (width 0.25) (layer "B.Cu") (net 0))
   (segment (start 297.0603 92.075) (end 295.2623 93.873) (width 0.2) (layer "B.Cu") (net 0))
@@
   (segment (start 143.3195 52.7685) (end 141.5415 54.5465) (width 0.25) (layer "B.Cu") (net 0))
   (segment (start 83.693 246.9515) (end 83.693 255.4605) (width 0.25) (layer "B.Cu") (net 0))
+  (segment (start 105.7275 124.206) (end 40.132 124.206) (width 0.6) (layer "B.Cu") (net 0))
   (segment (start 128.7145 27.305) (end 128.7145 52.07) (width 0.2) (layer "B.Cu") (net 0))
   (segment (start 184.7415 249.575) (end 185.9915 250.825) (width 0.25) (layer "B.Cu") (net 0))
@@
   (segment (start 96.393 202.692) (end 96.393 177.927) (width 0.25) (layer "B.Cu") (net 0))
   (segment (start 215.773 79.375) (end 217.063 79.375) (width 0.25) (layer "B.Cu") (net 0))
+  (segment (start 40.132 124.206) (end 40.132 117.856) (width 0.6) (layer "B.Cu") (net 0))
   (segment (start 329.2475 178.0975) (end 329.2475 141.9225) (width 0.25) (layer "B.Cu") (net 0))
   (segment (start 191.77 41.1045) (end 192.806 40.0685) (width 0.25) (layer "B.Cu") (net 0))
