File: Final Board/luminator/luminator.kicad_pcb (KiCad board)
At the start: 4 copper layers, 308.6 x 109.2 mm, 192 parts

Commit message: asd
Parts:
- removed the REF** at (327.0, 214.1)
- removed the REF** at (308.3, 202.1)
- removed the REF** at (334.9, 210.7)
- removed the REF** at (334.9, 161.2)
- removed the REF** at (322.9, 184.9)
- removed the REF** at (327.0, 189.4)
- removed the REF** at (322.9, 160.1)
- removed the REF** at (327.0, 164.6)
- removed the REF** at (334.9, 235.5)
- removed the REF** at (327.0, 139.8)
- removed the REF** at (338.8, 163.6)
- removed the REF** at (338.8, 213.9)
- removed the REF** at (338.6, 237.2)
- removed the REF** at (338.8, 188.5)
- removed the REF** at (348.3, 202.1)
- removed the REF** at (348.3, 235.7)
- removed the REF** at (308.3, 235.7)
- removed the REF** at (322.9, 209.7)
- removed the REF** at (322.9, 234.4)
- removed the REF** at (334.9, 185.9)
- added REF**: P78E05, Luminator:P78E05, F.Cu at (98.3, 118.1)
- added REF**: DS3231 RTC, Luminator:DS3231 RTC, F.Cu at (38.9, 64.4)
- added REF**: ESP-01, Luminator:ESP-01, F.Cu at (42.7, 90.8)
- added REF**: CP_Radial_D10.0mm_P5.00mm, Capacitor_THT:CP_Radial_D10.0mm_P5.00mm, F.Cu at (40.6, 106.2)
- added REF**: MODULE_ESP32_DEVKIT_V1, Luminator:MODULE_ESP32_DEVKIT_V1, F.Cu at (82.0, 85.6)
- added REF**: CP_Radial_D5.0mm_P2.50mm, Capacitor_THT:CP_Radial_D5.0mm_P2.50mm, F.Cu at (36.8, 125.3)
- added REF**: CONN_1729128_PXC, Luminator:CONN_1729128_PXC, F.Cu at (32.3, 101.1)
- XA**: moved to B.Cu
- moved XA** 52.1 mm to (51.6, 121.4)
- moved REF** 3.81 mm to (43.9, 117.9)
Routing:
- net (no net): track 35888.9 -> 33347.1 mm, vias 397 -> 377
Other:
- board size 308.6 x 109.2 mm -> 296.7 x 109.2 mm
- board text added: "+POS"
- board text added: "AVR ONLY"
- board text added: "Luminator Flipdot Controller Designed by Tyler Bowers, 2023"
- board text added: "NO AVR"
- board text added: "ROWS"
- board text removed: "Inner layers 1 and 2 are used for tran array outputs to connectors, outer layers are used for component signals."
- board text removed: "TODO: Power to tran array, serial order & conn"

Commit message: asd
Parts:
- removed the REF** at (42.7, 90.8)
- removed the XA** at (51.6, 121.4)
- added XA**: Arduino_Uno_R3_Shield, Luminator:Arduino_Uno_R3_Shield, B.Cu at (51.6, 121.4)
- moved REF** 29.1 mm to (54.1, 39.6), turned to -90 degrees
- moved REF** 20.2 mm to (47.9, 108.5), turned to 180 degrees
- moved REF** 19.5 mm to (42.2, 84.3)
- moved REF** 6.10 mm to (40.3, 100.1)
Routing:
- net (no net): track 33347.1 -> 33182.8 mm
Other:
- board size 296.7 x 109.2 mm -> 287.5 x 109.2 mm
- board text added: "#ARDUINO D2= D3= D4= D5= D6= D7= D8= D9= D10= D11= A4= A5= #ESP32"

Commit message: asd
Parts:
- removed the REF** at (90.0, 202.7)
- removed the REF** at (101.1, 248.7)
- removed the REF** at (182.1, 273.4)
- removed the REF** at (116.7, 227.5)
- removed the REF** at (137.1, 240.2)
- removed the REF** at (182.1, 199.1)
- removed the REF** at (170.1, 198.1)
- removed the REF** at (31.5, 201.7)
- removed the REF** at (39.4, 223.0)
- removed the REF** at (290.1, 120.7)
- removed the REF** at (86.0, 247.8)
- removed the REF** at (31.5, 176.9)
- removed the REF** at (112.6, 198.2)
- removed the REF** at (210.1, 120.7)
- removed the REF** at (112.6, 223.0)
- removed the REF** at (39.4, 198.2)
- removed the REF** at (174.2, 227.3)
- removed the REF** at (74.2, 174.5)
- removed the REF** at (78.1, 201.7)
- removed the REF** at (86.0, 272.5)
- removed the REF** at (86.0, 198.2)
- removed the REF** at (170.1, 272.4)
- removed the REF** at (250.1, 120.7)
- removed the REF** at (78.1, 251.2)
- removed the REF** at (78.1, 226.4)
- removed the REF** at (186.0, 201.5)
- removed the REF** at (39.4, 247.8)
- removed the REF** at (186.0, 251.8)
- removed the REF** at (104.8, 251.2)
- removed the REF** at (90.0, 227.5)
- removed the REF** at (78.1, 176.9)
- removed the REF** at (104.8, 201.7)
- removed the REF** at (174.2, 177.8)
- removed the REF** at (43.4, 177.9)
- removed the REF** at (101.1, 224.0)
- removed the REF** at (182.1, 248.7)
- removed the REF** at (74.2, 223.8)
- removed the REF** at (74.2, 248.7)
- removed the REF** at (116.7, 177.9)
- removed the REF** at (31.5, 226.4)
- removed the REF** at (90.0, 177.9)
- removed the REF** at (104.8, 176.9)
- removed the REF** at (112.6, 247.8)
- removed the REF** at (116.7, 252.2)
- removed the REF** at (100.9, 199.1)
- removed the REF** at (195.5, 273.7)
- removed the REF** at (186.0, 226.4)
- removed the REF** at (90.0, 252.2)
- removed the REF** at (195.5, 240.0)
- removed the REF** at (170.1, 247.7)
- removed the REF** at (185.8, 275.2)
- removed the REF** at (155.5, 240.0)
- removed the REF** at (86.0, 223.0)
- removed the REF** at (43.4, 227.5)
- removed the REF** at (31.5, 251.2)
- removed the REF** at (182.1, 223.9)
- removed the REF** at (39.4, 272.5)
- removed the REF** at (170.1, 222.9)
- removed the REF** at (27.6, 199.5)
- removed the REF** at (27.6, 174.8)
- removed the REF** at (100.9, 174.5)
- removed the REF** at (116.7, 202.7)
- removed the REF** at (74.2, 199.1)
- removed the REF** at (27.6, 224.3)
- removed the REF** at (112.6, 272.5)
- removed the REF** at (155.5, 273.7)
- removed the REF** at (27.6, 249.0)
- removed the REF** at (104.8, 226.4)
- removed the REF** at (43.4, 202.7)
- removed the REF** at (174.2, 202.6)
- removed the REF** at (43.4, 252.2)
- removed the REF** at (174.2, 252.1)
Routing:
- net (no net): track 33182.8 -> 23017.2 mm, vias 377 -> 205
Other:
- board text added: "#ARDUINO D2=R.Serial D3=R.OE D4=R.RCLK D5=R.SRCLK D6=R.SRCLR D7=C.Serial D8=C.OE D9=C.RCLK D10=C.SRCLK D11=C.SRCLR A4=RTC.SDA A5=RTC.SCL #ESP32 GPIO32=R.Serial GPIO33=R.OE GPIO25=R.RCLK GPIO26=R.SRCLK GPIO27=R.SRCLR GPIO36=C.Serial GPIO19=C.OE GPIO18=C.RCLK GPIO17=C.SRCLK GPIO16=C.SRCLR GPIO22=RTC.SCL GPIO21=RTC.SDA"
- board text added: "Luminator Flipdot Controller 16x112 Designed by Tyler Bowers, 2023"
- board text removed: "#ARDUINO D2= D3= D4= D5= D6= D7= D8= D9= D10= D11= A4= A5= #ESP32"
- board text removed: "+12/24V"
- board text removed: "+5V"
- board text removed: "3 4 1 2"
- board text removed: "COL 1-8"
- board text removed: "COL 17-24"
- board text removed: "COL 25-28(32)"
- board text removed: "COL 9-16"
- board text removed: "Luminator Flipdot Controller Designed by Tyler Bowers, 2023"
