File: final board/luminator.kicad_pcb (KiCad board)
At the start: 4 copper layers, 287.5 x 109.2 mm, 106 parts

Commit message: asd
Parts:
- removed the REF** at (240.5, 98.8)
- removed the REF** at (290.1, 120.7)
- removed the REF** at (188.7, 49.5)
- removed the REF** at (107.1, 95.5)
- removed the REF** at (111.1, 48.5)
- removed the REF** at (276.6, 70.9)
- removed the REF** at (40.3, 100.1)
- removed the REF** at (137.7, 98.0)
- removed the REF** at (107.1, 70.6)
- removed the REF** at (118.9, 119.4)
- removed the REF** at (250.1, 87.0)
- removed the REF** at (210.1, 120.7)
- removed the REF** at (196.6, 46.1)
- removed the REF** at (276.6, 120.4)
- removed the REF** at (268.7, 24.8)
- removed the REF** at (133.8, 46.0)
- removed the REF** at (276.6, 46.1)
- removed the REF** at (137.7, 73.3)
- removed the REF** at (240.5, 48.5)
- removed the REF** at (123.0, 74.3)
- removed the REF** at (304.7, 119.4)
- removed the REF** at (304.7, 69.8)
- removed the REF** at (200.5, 98.8)
- removed the REF** at (250.1, 120.7)
- removed the REF** at (280.5, 73.4)
- removed the REF** at (236.6, 70.9)
- removed the REF** at (268.7, 99.1)
- removed the REF** at (308.7, 49.5)
- removed the REF** at (224.7, 45.1)
- removed the REF** at (149.7, 49.5)
- removed the REF** at (111.1, 98.0)
- removed the REF** at (196.6, 70.9)
- removed the REF** at (82.0, 85.6)
- removed the REF** at (123.0, 49.5)
- removed the REF** at (236.6, 46.1)
- removed the REF** at (137.7, 23.7)
- removed the REF** at (188.7, 99.1)
- removed the REF** at (188.7, 74.3)
- removed the REF** at (145.6, 45.1)
- removed the REF** at (316.6, 120.4)
- removed the REF** at (145.6, 119.4)
- removed the REF** at (320.5, 98.8)
- removed the REF** at (228.7, 24.8)
- removed the REF** at (149.7, 24.8)
- removed the REF** at (264.7, 69.8)
- removed the REF** at (184.7, 94.6)
- removed the REF** at (134.1, 70.9)
- removed the REF** at (236.6, 120.4)
- removed the REF** at (149.7, 99.1)
- removed the REF** at (210.1, 87.0)
- removed the REF** at (200.5, 73.4)
- removed the REF** at (264.7, 45.1)
- removed the REF** at (184.7, 119.4)
- removed the REF** at (316.6, 46.1)
- removed the REF** at (107.1, 46.0)
- removed the REF** at (43.9, 117.9)
- removed the REF** at (308.7, 24.8)
- removed the REF** at (149.7, 74.3)
- removed the REF** at (280.5, 48.5)
- removed the REF** at (42.2, 84.3)
- removed the REF** at (224.7, 94.6)
- removed the REF** at (47.9, 108.5)
- removed the REF** at (137.7, 48.5)
- removed the REF** at (196.6, 95.6)
- removed the REF** at (280.5, 98.8)
- removed the REF** at (290.1, 87.0)
- removed the REF** at (276.6, 95.6)
- removed the REF** at (228.7, 74.3)
- removed the REF** at (316.6, 70.9)
- removed the REF** at (320.5, 73.4)
- removed the REF** at (320.5, 48.5)
- removed the REF** at (224.7, 69.8)
- removed the REF** at (240.5, 73.4)
- removed the REF** at (118.9, 45.1)
- removed the REF** at (123.0, 99.1)
- removed the REF** at (134.1, 95.5)
- removed the REF** at (184.7, 69.8)
- removed the REF** at (228.7, 49.5)
- removed the REF** at (196.6, 120.4)
- removed the REF** at (308.7, 74.3)
- removed the REF** at (316.6, 95.6)
- removed the REF** at (98.3, 118.1)
- removed the REF** at (145.6, 69.8)
- removed the REF** at (224.7, 119.4)
- removed the REF** at (264.7, 119.4)
- removed the REF** at (200.5, 48.5)
- removed the REF** at (308.7, 99.1)
- removed the REF** at (111.1, 23.7)
- removed the REF** at (188.7, 24.8)
- removed the REF** at (170.1, 120.7)
- removed the REF** at (264.7, 94.6)
- removed the REF** at (268.7, 49.5)
- removed the REF** at (54.1, 39.6)
- removed the REF** at (304.7, 94.6)
- removed the REF** at (228.7, 99.1)
- removed the REF** at (304.7, 45.1)
- removed the REF** at (123.0, 24.8)
- removed the REF** at (111.1, 73.3)
- removed the REF** at (118.9, 94.6)
- removed the REF** at (236.6, 95.6)
- removed the REF** at (268.7, 74.3)
- removed the REF** at (118.9, 69.8)
- removed the REF** at (184.7, 45.1)
- removed the REF** at (170.1, 87.0)
- removed the REF** at (145.6, 94.6)
- removed XA**: Arduino_Uno_R3_Shield, Luminator:Arduino_Uno_R3_Shield
- added REF**: SIP-14, Luminator:SIP-14, F.Cu at (124.0, 72.4)
- added REF**: SIP-14, Luminator:SIP-14, F.Cu at (106.4, 72.4)
- added REF**: TSSOP-28EP_MPQ6628_MNP, Luminator:TSSOP-28EP_MPQ6628_MNP, F.Cu at (115.2, 72.4)
Routing:
- net (no net): track 23017.2 -> 278.6 mm, vias 205 -> 0
Other:
- board size 287.5 x 109.2 mm -> 20.1 x 35.6 mm
- copper layers 4 -> 2
- board text added: "1"
- board text added: "14"
- board text added: "15"
- board text added: "24"
- board text added: "MPQ6628 Adapter"
- board text removed: "#ARDUINO D2=R.Serial D3=R.OE D4=R.RCLK D5=R.SRCLK D6=R.SRCLR D7=C.Serial D8=C.OE D9=C.RCLK D10=C.SRCLK D11=C.SRCLR A4=RTC.SDA A5=RTC.SCL #ESP32 GPIO32=R.Serial GPIO33=R.OE GPIO25=R.RCLK GPIO26=R.SRCLK GPIO27=R.SRCLR GPIO36=C.Serial GPIO19=C.OE GPIO18=C.RCLK GPIO17=C.SRCLK GPIO16=C.SRCLR GPIO22=RTC.SCL GPIO21=RTC.SDA"
- board text removed: "*"
- board text removed: "+POS"
- board text removed: "AVR ONLY"
- board text removed: "B1"
- board text removed: "B2"
- board text removed: "B3"
- board text removed: "B4"
- board text removed: "COLS"
- board text removed: "GND"
- board text removed: "Luminator Flipdot Controller 16x112 Designed by Tyler Bowers, 2023"
- board text removed: "NO AVR"
- board text removed: "ROWS"

Commit message: asd
Parts:
- removed the REF** at (124.0, 72.4)
- removed the REF** at (106.4, 72.4)
- added REF**: M HEADER 2x25=50, Luminator:M HEADER 2x25=50 2.54mm, F.Cu at (126.0, 95.0)
- added REF**: M HEADER 2x25=50, Luminator:M HEADER 2x25=50 2.54mm, F.Cu at (150.1, 95.0)
- added REF**: M HEADER 2x25=50, Luminator:M HEADER 2x25=50 2.54mm, F.Cu at (174.2, 95.0)
- added REF**: M HEADER 2x25=50, Luminator:M HEADER 2x25=50 2.54mm, F.Cu at (101.9, 95.0)
- added REF**: MODULE_ESP32_DEVKIT_V1, Luminator:MODULE_ESP32_DEVKIT_V1, F.Cu at (51.8, 69.6)
- moved REF** 33.0 mm to (90.4, 50.5)
Routing:
- net (no net): track 278.6 -> 0.00 mm
Other:
- board outline removed
- board text removed: "1"
- board text removed: "14"
- board text removed: "15"
- board text removed: "24"
- board text removed: "MPQ6628 Adapter"

Commit message: asd
Parts:
- removed the REF** at (126.0, 95.0)
- removed the REF** at (150.1, 95.0)
- removed the REF** at (174.2, 95.0)
- added REF**: M HEADER 2x10=20, Luminator:M HEADER 2x10=20 2.54mm, F.Cu at (101.9, 131.3)
- added REF**: DS3231 RTC, Luminator:DS3231 RTC, F.Cu at (73.9, 40.9)
- added REF**: TSSOP-28EP_MPQ6628_MNP, Luminator:TSSOP-28EP_MPQ6628_MNP, F.Cu at (111.3, 119.9)
- moved REF** 25.2 mm to (111.4, 64.5)
- moved REF** 14.3 mm to (50.3, 83.8)
Routing:
- net (no net): track 0.00 -> 52.9 mm
Other:
- board text added: "*"

Commit message: asd
Routing:
- net (no net): track 52.9 -> 141.6 mm
Changed lines of the file:
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@@
   )
   (footprint "Luminator:TSSOP-28EP_MPQ6628_MNP" (layer "F.Cu")
-    (at 111.252 119.888 90)
+    (at 111.261499 119.888 90)
     (tags "MPQ6628GF-AEC1-P ")
     (attr smd)
@@
     (effects (font (size 1 1) (thickness 0.15)))
   )
+  (segment (start 114.836498 119.888) (end 114.836498 122.809) (width 0.4) (layer "F.Cu") (net 0))
+  (segment (start 114.186499 114.567499) (end 109.347 109.728) (width 0.4) (layer "F.Cu") (net 0))
   (segment (start 99.314 126.238) (end 101.854 126.238) (width 0.4) (layer "F.Cu") (net 0))
   (segment (start 101.854 89.916) (end 100.584 88.646) (width 0.4) (layer "F.Cu") (net 0))
+  (segment (start 108.336499 124.835501) (end 108.336499 122.809) (width 0.4) (layer "F.Cu") (net 0))
+  (segment (start 107.6865 119.888) (end 107.6865 116.967) (width 0.4) (layer "F.Cu") (net 0))
   (segment (start 101.854 54.356) (end 101.854 51.816) (width 0.4) (layer "F.Cu") (net 0))
   (segment (start 99.314 110.998) (end 101.854 110.998) (width 0.4) (layer "F.Cu") (net 0))
@@
   (segment (start 101.854 123.698) (end 99.314 123.698) (width 0.4) (layer "F.Cu") (net 0))
   (segment (start 99.314 116.078) (end 101.854 116.078) (width 0.4) (layer "F.Cu") (net 0))
+  (segment (start 114.836498 116.967) (end 114.836498 119.888) (width 0.4) (layer "F.Cu") (net 0))
   (segment (start 101.854 56.896) (end 101.854 59.436) (width 0.4) (layer "F.Cu") (net 0))
+  (segment (start 109.347 109.728) (end 98.298 109.728) (width 0.4) (layer "F.Cu") (net 0))
   (segment (start 101.854 41.656) (end 100.584 42.926) (width 0.4) (layer "F.Cu") (net 0))
   (segment (start 101.854 113.538) (end 99.314 113.538) (width 0.4) (layer "F.Cu") (net 0))
+  (segment (start 97.79 112.903) (end 97.79 127.254) (width 0.4) (layer "F.Cu") (net 0))
   (segment (start 101.854 61.976) (end 101.854 64.516) (width 0.4) (layer "F.Cu") (net 0))
+  (segment (start 108.336499 116.967) (end 108.336499 115.448499) (width 0.4) (layer "F.Cu") (net 0))
+  (segment (start 111.5865 116.967) (end 111.5865 119.562999) (width 0.4) (layer "F.Cu") (net 0))
   (segment (start 101.854 77.216) (end 101.854 79.756) (width 0.4) (layer "F.Cu") (net 0))
   (segment (start 99.314 121.158) (end 101.854 121.158) (width 0.4) (layer "F.Cu") (net 0))
   (segment (start 101.854 128.778) (end 99.314 128.778) (width 0.4) (layer "F.Cu") (net 0))
+  (segment (start 105.156 112.268) (end 98.425 112.268) (width 0.4) (layer "F.Cu") (net 0))
   (segment (start 100.584 45.466) (end 101.854 46.736) (width 0.4) (layer "F.Cu") (net 0))
+  (segment (start 114.186499 116.967) (end 114.186499 114.567499) (width 0.4) (layer "F.Cu") (net 0))
+  (segment (start 108.336499 115.448499) (end 105.156 112.268) (width 0.4) (layer "F.Cu") (net 0))
   (segment (start 101.854 67.056) (end 101.854 69.596) (width 0.4) (layer "F.Cu") (net 0))
+  (segment (start 114.836498 119.888) (end 111.261499 119.888) (width 0.4) (layer "F.Cu") (net 0))
   (segment (start 100.584 42.926) (end 100.584 45.466) (width 0.4) (layer "F.Cu") (net 0))
   (segment (start 101.854 108.458) (end 99.314 108.458) (width 0.4) (layer "F.Cu") (net 0))
+  (segment (start 98.425 112.268) (end 97.79 112.903) (width 0.4) (layer "F.Cu") (net 0))
+  (segment (start 101.854 131.318) (end 108.336499 124.835501) (width 0.4) (layer "F.Cu") (net 0))
+  (segment (start 112.236498 118.913001) (end 111.261499 119.888) (width 0.4) (layer "F.Cu") (net 0))
   (segment (start 100.584 86.106) (end 101.854 84.836) (width 0.4) (layer "F.Cu") (net 0))
+  (segment (start 111.5865 119.562999) (end 111.261499 119.888) (width 0.4) (layer "F.Cu") (net 0))
   (segment (start 101.854 131.318) (end 99.314 131.318) (width 0.4) (layer "F.Cu") (net 0))
   (segment (start 100.584 88.646) (end 100.584 86.106) (width 0.4) (layer "F.Cu") (net 0))
   (segment (start 101.854 118.618) (end 99.314 118.618) (width 0.4) (layer "F.Cu") (net 0))
+  (segment (start 97.79 127.254) (end 99.314 128.778) (width 0.4) (layer "F.Cu") (net 0))
+  (segment (start 112.236498 116.967) (end 112.236498 118.913001) (width 0.4) (layer "F.Cu") (net 0))
+  (segment (start 98.298 109.728) (end 97.028 110.998) (width 0.4) (layer "F.Cu") (net 0))
+  (segment (start 107.6865 119.888) (end 111.261499 119.888) (width 0.4) (layer "F.Cu") (net 0))
+  (segment (start 107.6865 122.809) (end 107.6865 119.888) (width 0.4) (layer "F.Cu") (net 0))
 )

Commit message: asd
Parts:
- moved REF** 0.29 mm to (111.5, 119.8)
Routing:
- net (no net): track 141.6 -> 225.3 mm, vias 0 -> 4

Commit message: asd
Parts:
- turned REF** to 90 degrees
Routing:
- net (no net): track 225.3 -> 392.2 mm, vias 4 -> 7

Commit message: asd
Parts:
- added REF**: M HEADER 2x10=20, Luminator:M HEADER 2x10=20 2.54mm, F.Cu at (167.5, 131.3)
- added REF**: TSSOP-28EP_MPQ6628_MNP, Luminator:TSSOP-28EP_MPQ6628_MNP, F.Cu at (155.1, 64.5)
- added REF**: TSSOP-28EP_MPQ6628_MNP, Luminator:TSSOP-28EP_MPQ6628_MNP, F.Cu at (133.4, 119.8)
- added REF**: TSSOP-28EP_MPQ6628_MNP, Luminator:TSSOP-28EP_MPQ6628_MNP, F.Cu at (89.7, 55.4)
- added REF**: TSSOP-28EP_MPQ6628_MNP, Luminator:TSSOP-28EP_MPQ6628_MNP, F.Cu at (155.3, 119.8)
- added REF**: M HEADER 2x10=20, Luminator:M HEADER 2x10=20 2.54mm, F.Cu at (123.7, 131.3)
- added REF**: M HEADER 2x25=50, Luminator:M HEADER 2x25=50 2.54mm, F.Cu at (167.5, 95.0)
- added REF**: TSSOP-28EP_MPQ6628_MNP, Luminator:TSSOP-28EP_MPQ6628_MNP, F.Cu at (176.9, 64.4)
- added REF**: M HEADER 2x25=50, Luminator:M HEADER 2x25=50 2.54mm, F.Cu at (123.7, 95.0)
- added REF**: M HEADER 2x25=50, Luminator:M HEADER 2x25=50 2.54mm, F.Cu at (145.6, 95.0)
- added REF**: TSSOP-28EP_MPQ6628_MNP, Luminator:TSSOP-28EP_MPQ6628_MNP, F.Cu at (133.3, 64.5)
- added REF**: TSSOP-28EP_MPQ6628_MNP, Luminator:TSSOP-28EP_MPQ6628_MNP, F.Cu at (89.7, 72.5)
- added REF**: M HEADER 2x10=20, Luminator:M HEADER 2x10=20 2.54mm, F.Cu at (145.6, 131.3)
- added REF**: TSSOP-28EP_MPQ6628_MNP, Luminator:TSSOP-28EP_MPQ6628_MNP, F.Cu at (89.7, 89.6)
- added REF**: TSSOP-28EP_MPQ6628_MNP, Luminator:TSSOP-28EP_MPQ6628_MNP, F.Cu at (89.7, 39.6)
- added REF**: TSSOP-28EP_MPQ6628_MNP, Luminator:TSSOP-28EP_MPQ6628_MNP, F.Cu at (177.1, 119.7)
- moved REF** 34.4 mm to (62.0, 73.2), turned to 0 degrees
- moved REF** 31.0 mm to (64.8, 111.3)
Routing:
- net (no net): track 392.2 -> 4674.2 mm, vias 7 -> 60
Other:
- copper layers 2 -> 4
