File: final board/luminator.kicad_pcb (KiCad board)
At the start: 4 copper layers, 22 parts

Commit message: asd
Routing:
- net (no net): track 4674.2 -> 5406.6 mm, vias 60 -> 88
Other:
- board text added: "12-24v"
- board text added: "CLK"
- board text added: "CS_c1"
- board text added: "CS_c2"
- board text added: "CS_c3"
- board text added: "CS_c4"
- board text added: "DI"
- board text added: "DO"
- board text added: "EN"
- board text added: "GND"
- board text added: "VCC 5v"

Commit message: asd
Routing:
- net (no net): track 5406.6 -> 6102.4 mm, vias 88 -> 98
Other:
- board text added: "CS_r1.1"

Commit message: asd
Parts:
- added PS**: R78K5020, Luminator:R78K5020, F.Cu at (85.3, 119.5)
- added REF**: PHOENIX_1729128, Luminator:PHOENIX_1729128, F.Cu at (88.0, 132.6)
- added REF**: 0.1uF Ceramic, Luminator:0.1uF Ceramic, F.Cu at (78.6, 68.3)
- added REF**: CAP_YX_12P5X20_RUB, Luminator:CAP_YX_12P5X20_RUB, F.Cu at (85.2, 110.2)
- added REF**: SN74AHC595N, Luminator:SN74AHC595N, F.Cu at (34.6, 84.1)
Routing:
- net (no net): track 6102.4 -> 8077.3 mm, vias 98 -> 173
Other:
- board text added: "CS_r1.2"
- board text added: "VIN"

Commit message: asd
Parts:
- added REF**: CP_Radial_D5.0mm_P2.00mm, Capacitor_THT:CP_Radial_D5.0mm_P2.00mm, F.Cu at (78.9, 87.8)
- added REF**: 0.1uF Ceramic, Luminator:0.1uF Ceramic, F.Cu at (80.3, 56.7)
- added REF**: 0.1uF Ceramic, Luminator:0.1uF Ceramic, F.Cu at (158.5, 81.5)
- added REF**: 0.1uF Ceramic, Luminator:0.1uF Ceramic, F.Cu at (136.6, 81.6)
- added REF**: SN74AHC595N, Luminator:SN74AHC595N, F.Cu at (91.0, 108.0)
- added REF**: 0.1uF Ceramic, Luminator:0.1uF Ceramic, F.Cu at (114.7, 81.5)
- added REF**: 0.1uF Ceramic, Luminator:0.1uF Ceramic, F.Cu at (180.3, 81.5)
- moved REF** 65.3 mm to (52.0, 78.1), turned to -90 degrees
- moved REF** 52.4 mm to (81.3, 108.0)
- moved PS** 48.6 mm to (65.2, 75.3), turned to -90 degrees
- moved REF** 36.3 mm to (74.8, 75.4), turned to -90 degrees
- moved REF** 27.8 mm to (80.3, 40.6)
- moved REF** 5.93 mm to (59.3, 67.9)
- moved REF** 2.45 mm to (62.4, 111.0)
Routing:
- net (no net): track 8077.3 -> 8843.6 mm, vias 173 -> 179
Other:
- board text added: "CS_r2.1"
- board text added: "CS_r2.2"
- board text added: "CS_r3.1"
- board text added: "CS_r3.2"
- board text added: "CS_r4.1"
- board text added: "CS_r4.2"

Commit message: asd
Parts:
- added REF**: 0.1uF Ceramic, Luminator:0.1uF Ceramic, F.Cu at (174.7, 106.4)
- added REF**: 0.1uF Ceramic, Luminator:0.1uF Ceramic, F.Cu at (152.9, 106.4)
- added REF**: LED_D3.0mm, Luminator:LED_D3.0mm, F.Cu at (73.5, 65.8)
- added REF**: 0.1uF Ceramic, Luminator:0.1uF Ceramic, F.Cu at (80.4, 70.5)
- added REF**: 0.1uF Ceramic, Luminator:0.1uF Ceramic, F.Cu at (131.0, 106.4)
- added REF**: LED_D3.0mm, Luminator:LED_D3.0mm, F.Cu at (73.5, 57.4)
- added REF**: 0.1uF Ceramic, Luminator:0.1uF Ceramic, F.Cu at (109.2, 106.8)
Routing:
- net (no net): track 8843.6 -> 9263.1 mm
Other:
- board outline added: 138.6 x 109.3 mm
- board text added: "12-24V"
- board text added: "5V"

Commit message: asd
Parts:
- added REF**: ESP8266, Luminator:ESP8266, F.Cu at (60.6, 108.8)
- added REF**: R_Axial_DIN0207_L6.3mm_D2.5mm_P10.16mm_Horizontal, Resistor_THT:R_Axial_DIN0207_L6.3mm_D2.5mm_P10.16mm_Horizontal, F.Cu at (76.5, 69.0)
- added REF**: R_Axial_DIN0207_L6.3mm_D2.5mm_P10.16mm_Horizontal, Resistor_THT:R_Axial_DIN0207_L6.3mm_D2.5mm_P10.16mm_Horizontal, F.Cu at (72.9, 69.0)
- REF**: value MODULE_ESP32_DEVKIT_V1 -> ESP32 DEVKIT V1
- moved REF** 12.0 mm to (73.4, 45.4)
- moved REF** 12.0 mm to (73.5, 53.8)
- moved REF** 0.32 mm to (52.0, 77.8)
Routing:
- net (no net): track 9263.1 -> 9394.6 mm
Other:
- board text added: "10k"
- board text added: "Luminator Flipdot Controller 16x112 Designed in 2023 by Tyler Bowers"
- board text added: "MPQ6628GF"
- board text added: "Tylerebowers.com"

Commit message: asd
Parts:
- added REF**: 0.1uF Ceramic, Luminator:0.1uF Ceramic, F.Cu at (78.9, 96.8)
- added REF**: R_Axial_DIN0207_L6.3mm_D2.5mm_P10.16mm_Horizontal, Resistor_THT:R_Axial_DIN0207_L6.3mm_D2.5mm_P10.16mm_Horizontal, F.Cu at (88.2, 130.5)
- added REF**: LED_D3.0mm, Luminator:LED_D3.0mm, F.Cu at (94.6, 134.5)
- added REF**: LED_D3.0mm, Luminator:LED_D3.0mm, F.Cu at (84.9, 134.5)
- added REF**: LED_D3.0mm, Luminator:LED_D3.0mm, F.Cu at (89.7, 134.5)
- added REF**: LED_D3.0mm, Luminator:LED_D3.0mm, F.Cu at (80.1, 134.5)
- added REF**: 0.1uF Ceramic, Luminator:0.1uF Ceramic, F.Cu at (93.7, 130.5)
Routing:
- net (no net): track 9394.6 -> 9563.6 mm, vias 179 -> 170
